File: pcb/Axis_V1/Axis_V1.kicad_pcb (KiCad board)
At the start: 2 copper layers, 35 parts, among them J1 Screw_Terminal_01x03, J10 BOILER_3v3, J11 3WAY_L, J2 Screw_Terminal_01x03, J3 BREW_SW, J4 STEAM_SW, J5 AC_L, J6 AC_N, J7 BOILER_GND, J9 PUMP_L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

Commit message: Updates, add Pico MCU from github
Parts:
- moved U3 105.2 mm to (203.2, 68.7)
- moved J4 93.1 mm to (202.1, 106.7)
- moved U2 84.5 mm to (173.0, 117.0)
- moved J3 83.3 mm to (202.1, 100.1)
- moved C1 78.3 mm to (203.6, 90.8)
- moved R6 77.6 mm to (203.4, 74.5)
- moved J11 61.3 mm to (202.7, 64.4)
- moved R10 60.3 mm to (191.3, 90.1)
- moved TC1 59.1 mm to (114.3, 96.5)
- moved Q2 56.0 mm to (198.9, 81.8), turned to 0 degrees
- moved Q3 54.8 mm to (198.9, 87.7), turned to 0 degrees
- moved J2 53.6 mm to (142.2, 94.0), turned to 0 degrees
- moved C3 53.4 mm to (203.6, 94.7)
- moved R11 49.2 mm to (191.3, 95.0), turned to 0 degrees
- moved OC3 48.3 mm to (165.1, 94.0)
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Other:
- board outline added: 101.6 x 55.9 mm

Commit message: Changes
Parts:
- OC1, OC2, OC3: footprint Package_DIP:DIP-6_W7.62mm -> Package_DIP:DIP-6_W7.62mm_LongPads
- R1: footprint Resistor_SMD:R_0805_2012Metric -> Resistor_SMD:R_1206_3216Metric
- moved U3 88.7 mm to (116.8, 88.9)
- moved J10 45.0 mm to (247.7, 62.1)
- moved J11 45.0 mm to (247.7, 64.4)
- moved J7 45.0 mm to (247.7, 57.5)
- moved J9 45.0 mm to (247.7, 59.8)
- moved R3 44.0 mm to (166.2, 88.9)
- moved D1 39.9 mm to (189.2, 92.7), turned to 90 degrees
- moved U2 39.8 mm to (144.8, 88.9)
- moved J3 39.6 mm to (162.6, 101.6)
- moved C1 37.9 mm to (166.4, 83.3), turned to 90 degrees
- moved R2 37.3 mm to (171.4, 81.3)
- moved C2 34.5 mm to (187.5, 62.2), turned to 180 degrees
- moved J4 32.4 mm to (170.2, 101.6)
- moved OC2 32.2 mm to (176.5, 54.6)
- moved R7 30.4 mm to (199.4, 55.9)
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
Commit message: Yepp
Parts:
- moved C1 3.81 mm to (166.4, 87.2)
- moved D1 3.81 mm to (189.2, 96.5)
- moved OC1 3.81 mm to (184.2, 94.0)
- moved Q1 3.81 mm to (170.2, 91.4)
- moved R2 3.81 mm to (171.4, 85.1)
- moved R6 3.81 mm to (195.6, 94.0)
- moved R3 3.81 mm to (166.2, 92.7)
- moved J4 1.27 mm to (170.2, 100.3)
Changed lines of the file:
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@@
   )
   (footprint "Resistor_SMD:R_1206_3216Metric" (layer "F.Cu")
-    (at 166.1775 88.9)
+    (at 166.1775 92.71)
     (descr "Resistor SMD 1206 (3216 Metric), square (rectangular) end terminal, IPC_7351 nominal, (Body size source: IPC-SM-782 page 72, https://www.pcb-3d.com/wordpress/wp-content/uploads/ipc-sm-782a_amendment_1_and_2.pdf), generated with kicad-footprint-generator")
     (tags "resistor")
@@
   )
   (footprint "Package_DIP:DIP-6_W7.62mm_LongPads" (layer "F.Cu")
-    (at 184.165 90.155 180)
+    (at 184.165 93.965 180)
     (descr "6-lead though-hole mounted DIP package, row spacing 7.62 mm (300 mils), LongPads")
     (tags "THT DIP DIL PDIP 2.54mm 7.62mm 300mil LongPads")
@@
   )
   (footprint "LED_SMD:LED_2512_6332Metric" (layer "F.Cu")
-    (at 195.58 90.17 -90)
+    (at 195.58 93.98 -90)
     (descr "LED SMD 2512 (6332 Metric), square (rectangular) end terminal, IPC_7351 nominal, (Body size source: http://www.tortai-tech.com/upload/download/2011102023233369053.pdf), generated with kicad-footprint-generator")
     (tags "LED")
@@
   )
   (footprint "Package_TO_SOT_THT:TO-92_Inline" (layer "F.Cu")
-    (at 170.18 87.63)
+    (at 170.18 91.44)
     (descr "TO-92 leads in-line, narrow, oval pads, drill 0.75mm (see NXP sot054_po.pdf)")
     (tags "to-92 sc-43 sc-43a sot54 PA33 transistor")
@@
   )
   (footprint "Connector_JST:JST_PH_B2B-PH-K_1x02_P2.00mm_Vertical" (layer "F.Cu")
-    (at 170.18 101.6)
+    (at 170.18 100.33)
     (descr "JST PH series connector, B2B-PH-K (http://www.jst-mfg.com/product/pdf/eng/ePH.pdf), generated with kicad-footprint-generator")
     (tags "connector JST PH side entry")
@@
   )
   (footprint "Diode_THT:D_DO-41_SOD81_P10.16mm_Horizontal" (layer "F.Cu")
-    (at 189.23 92.71 90)
+    (at 189.23 96.52 90)
     (descr "Diode, DO-41_SOD81 series, Axial, Horizontal, pin pitch=10.16mm, , length*diameter=5.2*2.7mm^2, , http://www.diodes.com/_files/packages/DO-41%20(Plastic).pdf")
     (tags "Diode DO-41_SOD81 series Axial Horizontal pin pitch 10.16mm  length 5.2mm diameter 2.7mm")
@@
   )
   (footprint "Capacitor_SMD:C_0402_1005Metric" (layer "F.Cu")
-    (at 166.37 83.34 90)
+    (at 166.37 87.15 90)
     (descr "Capacitor SMD 0402 (1005 Metric), square (rectangular) end terminal, IPC_7351 nominal, (Body size source: IPC-SM-782 page 76, https://www.pcb-3d.com/wordpress/wp-content/uploads/ipc-sm-782a_amendment_1_and_2.pdf), generated with kicad-footprint-generator")
     (tags "capacitor")
@@
   )
   (footprint "Resistor_SMD:R_1206_3216Metric" (layer "F.Cu")
-    (at 171.45 81.28)
+    (at 171.45 85.09)
     (descr "Resistor SMD 1206 (3216 Metric), square (rectangular) end terminal, IPC_7351 nominal, (Body size source: IPC-SM-782 page 72, https://www.pcb-3d.com/wordpress/wp-content/uploads/ipc-sm-782a_amendment_1_and_2.pdf), generated with kicad-footprint-generator")
     (tags "resistor")

Commit message: Add more stuff for pcb
Parts:
- removed C1: 100nF, Capacitor_SMD:C_0402_1005Metric
- D1: value 1N4001 -> RFN1LAM6STR; footprint Diode_THT:D_DO-41_SOD81_P10.16mm_Horizontal -> Diode_SMD:D_SOD-128
- OC1: footprint Package_DIP:DIP-6_W7.62mm_LongPads -> DIP:SMDIP-6_W7.62mm
- OC2, OC3: value MOC3021M -> MOC3021S-TA1; footprint Package_DIP:DIP-6_W7.62mm_LongPads -> DIP:SMDIP-6_W7.62mm
- Q2, Q3: footprint Package_TO_SOT_THT:TO-220-3_Vertical -> Package_TO_SOT_SMD:TO-252-2
- moved J7 102.9 mm to (145.4, 46.4)
- moved J10 93.4 mm to (155.6, 46.4)
- moved J11 39.4 mm to (211.5, 80.0)
- moved J9 36.4 mm to (211.5, 63.5)
- moved J5 18.4 mm to (211.5, 48.3)
- moved J4 14.2 mm to (156.2, 102.9)
- moved J1 14.0 mm to (130.8, 100.3)
- moved J2 14.0 mm to (113.0, 100.3)
- moved J3 14.0 mm to (148.6, 102.9)
- moved J6 11.8 mm to (211.5, 54.0)
- moved C2 11.7 mm to (196.2, 54.5), turned to 90 degrees
- moved TC1 11.5 mm to (115.6, 90.2)
- moved U2 9.71 mm to (135.3, 90.8)
- moved U3 9.67 mm to (125.7, 85.1)
- moved OC1 6.54 mm to (178.4, 90.8)
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Connections:
- OC1 pad 5: +3.3V -> unconnected-(OC1-Pad5)
- OC1 pad 6: unconnected-(OC1-Pad6) -> +3.3V
- U3 pad 5: PIN_10 -> PIN_12
- U3 pad 7: PIN_12 -> PIN_10
Other:
- board size 101.6 x 55.9 mm -> 108 x 63.5 mm

Commit message: PCB Updates
Parts:
- removed C2, C3: 100nF, Capacitor_SMD:C_0402_1005Metric
- removed D1: RFN1LAM6STR, Diode_SMD:D_SOD-128
- removed OC1: 4N35, DIP:SMDIP-6_W7.62mm
- removed OC2, OC3: MOC3021S-TA1, DIP:SMDIP-6_W7.62mm
- removed Q1: BC547, Package_TO_SOT_THT:TO-92_Inline
- removed Q2, Q3: BT136-500, Package_TO_SOT_SMD:TO-252-2
- removed R1, R8: 200, Resistor_SMD:R_1206_3216Metric
- removed R10, R5: 180, Resistor_SMD:R_2512_6332Metric
- removed R11, R7: 2.4k, Resistor_SMD:R_2512_6332Metric
- removed R2: 1M, Resistor_SMD:R_1206_3216Metric
- removed R3: 1k, Resistor_SMD:R_1206_3216Metric
- removed R4, R9: 100, Resistor_SMD:R_1206_3216Metric
- removed R6: 10k, LED_SMD:LED_2512_6332Metric

Commit message: More pcb updates
Parts:
- added C1: C_Small, Capacitor_SMD:C_1206_3216Metric, F.Cu at (186.3, 102.9)
- added C2: C_Small, Capacitor_SMD:C_1206_3216Metric, F.Cu at (182.2, 85.1)
- added D1: RFN1LAM6STR, Diode_SMD:D_SOD-128, F.Cu at (174.6, 24.8)
- added H1: MountingHole, MountingHole:MountingHole_2.7mm_M2.5, F.Cu at (95.9, 72.4)
- added H2: MountingHole, MountingHole:MountingHole_2.7mm_M2.5, F.Cu at (95.9, 116.8)
- added H3: MountingHole, MountingHole:MountingHole_2.7mm_M2.5, F.Cu at (197.5, 116.8)
- added H4: MountingHole, MountingHole:MountingHole_2.7mm_M2.5, F.Cu at (197.5, 72.4)
- added OC1: 4N35, Package_DIP:SMDIP-6_W7.62mm, F.Cu at (166.4, 24.8)
- added OC2: MOC3021S-TA1, Package_DIP:SMDIP-6_W7.62mm, F.Cu at (156.8, 40.0)
- added OC3: MOC3021S-TA1, Package_DIP:SMDIP-6_W7.62mm, F.Cu at (156.8, 53.3)
- added Q1: BC547, Package_TO_SOT_THT:TO-92_Inline, F.Cu at (152.4, 24.8)
- added Q2: BT136S-600, Package_TO_SOT_SMD:TO-252-2, F.Cu at (178.7, 75.8)
- added Q3: BT136S-600, Package_TO_SOT_SMD:TO-252-2, F.Cu at (179.4, 113.0)
- added R1: 470, Resistor_SMD:R_0201_0603Metric, F.Cu at (141.0, 76.2)
- added R10: 220, Resistor_SMD:R_2512_6332Metric, F.Cu at (179.3, 102.9)
- added R11: 470, Resistor_SMD:R_2512_6332Metric, F.Cu at (170.8, 47.6)
- added R2: 10k, Resistor_SMD:R_0201_0603Metric, F.Cu at (143.5, 76.2)
- added R4: 240, Resistor_SMD:R_0201_0603Metric, F.Cu at (149.2, 37.5)
- added R5: 470, Resistor_SMD:R_2512_6332Metric, F.Cu at (170.8, 34.3)
- added R6: 10k, Resistor_SMD:R_2512_6332Metric, F.Cu at (180.3, 24.8)
- added R7: 220, Resistor_SMD:R_2512_6332Metric, F.Cu at (175.3, 85.7)
- added R8: 470, Resistor_SMD:R_1206_3216Metric, F.Cu at (133.3, 74.3)
- added R9: 240, Resistor_SMD:R_1206_3216Metric, F.Cu at (148.0, 52.9)
- J1: value Screw_Terminal_01x03 -> TRANSDUCER
- moved TC1 135.5 mm to (246.7, 124.4), turned to 0 degrees
- moved J2 135.4 mm to (248.3, 94.6)
- moved J1 119.0 mm to (248.3, 81.6)
- moved J3 91.5 mm to (238.2, 121.7)
- moved J4 85.8 mm to (238.2, 128.2)
- moved J7 38.2 mm to (116.8, 71.8)
- moved J11 32.8 mm to (194.3, 108.0)
- moved U1 31.2 mm to (119.4, 89.5)
- moved J6 30.1 mm to (189.9, 74.9)
- moved J5 30.0 mm to (214.6, 78.1)
- moved J10 27.9 mm to (144.1, 71.8)
- moved U3 23.5 mm to (131.4, 107.9), turned to 90 degrees
- moved J9 22.9 mm to (189.9, 71.1)
- moved U2 18.2 mm to (142.9, 107.3), turned to 90 degrees
Connections:
- net ADC_IN renamed /ADC_IN
- net Net-(J1-Pin_1) renamed /PRES_SENS
- net Net-(TC1-+) renamed /POS_THCPL
- net Net-(TC1--) renamed /NEG_THCPL
- net PIN_10 renamed /MAX_SO
- net PIN_11 renamed /MAX_CS
- net PIN_12 renamed /MAX_SCL
- net PIN_18 renamed /BOILER_GPIO
- net PIN_21 renamed /STEAM_SW
- net PIN_22 renamed /BREW_SW
- J5 pad 1: LINE -> /AC_L
- J6 pad 1: NEUT -> /AC_N
- U1 pad 17: PIN_13 -> unconnected-(U1-GPIO13-Pad17)
- U1 pad 19: PIN_14 -> /ADS_SDA
- U1 pad 20: PIN_15 -> /ADS_SCL
- U1 pad 21: PIN_16 -> /ZC_SIGNAL
- U1 pad 22: PIN_17 -> /PUMP_GPIO
- U1 pad 25: PIN_19 -> /3WAY_GPIO
- U2 pad 10: PIN_15 -> /ADS_SDA
- U2 pad 2: PIN_13 -> unconnected-(U2-ALERT/RDY-Pad2)
- U2 pad 9: PIN_14 -> /ADS_SCL
Other:
- board size 108 x 63.5 mm -> 108 x 50.8 mm

Commit message: We're basically there, going to get BOM together.
Parts:
- removed J10: BOILER_3v3, Library:Quick Disconnect
- removed TC1: Thermocouple_Block, TerminalBlock_RND:TerminalBlock_RND_205-00232_1x02_P5.08mm_Horizontal
- added J8: Screw_Terminal_01x02, TerminalBlock_MetzConnect:TerminalBlock_MetzConnect_Type101_RT01602HBWC_1x02_P5.08mm_Horizontal, F.Cu at (118.9, 120.6)
- added R12: 100, Resistor_SMD:R_1206_3216Metric, F.Cu at (123.2, 73.5)
- added R3: 100, Resistor_SMD:R_1206_3216Metric, F.Cu at (128.3, 73.5)
- C1, C2: value C_Small -> 10nf
- J2: footprint TerminalBlock_MetzConnect:TerminalBlock_MetzConnect_Type073_RT02603HBLU_1x03_P5.08mm_Horizontal -> Connector_JST:JST_PH_B3B-PH-K_1x03_P2.00mm_Vertical
- J7: value BOILER_GND -> BOILER_SSR; footprint Library:Quick Disconnect -> Connector_JST:JST_PH_B2B-PH-K_1x02_P2.00mm_Vertical
- R1, R2, R4: footprint Resistor_SMD:R_0201_0603Metric -> Resistor_SMD:R_1206_3216Metric
- moved J2 149.4 mm to (101.6, 66.5)
- moved J3 138.8 mm to (110.9, 66.5)
- moved J4 134.9 mm to (118.2, 66.5)
- moved J1 121.3 mm to (133.1, 119.6)
- moved R6 91.8 mm to (154.9, 113.0), turned to 90 degrees
- moved D1 89.0 mm to (159.5, 112.5)
- moved OC1 73.6 mm to (156.9, 97.8), turned to 90 degrees
- moved R5 69.7 mm to (166.1, 103.8), turned to -90 degrees
- moved Q1 64.2 mm to (154.5, 89.0), turned to 0 degrees
- moved R11 57.7 mm to (183.8, 103.8), turned to -90 degrees
- moved OC2 55.1 mm to (166.6, 94.2), turned to -90 degrees
- moved H4 51.9 mm to (201.7, 124.2)
- moved H1 51.8 mm to (93.5, 124.2)
- moved H3 50.3 mm to (201.7, 66.8)
- moved H2 50.1 mm to (93.5, 66.8)
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Connections:
- net Net-(J11-Pin_1) renamed /3WAY_L
- net Net-(J9-Pin_1) renamed /PUMP_L
- J3 pad 1: +3.3V -> Net-(J3-Pin_1)
- J3 pad 2: /BREW_SW -> +3.3V
- J4 pad 1: +3.3V -> Net-(J4-Pin_1)
- J4 pad 2: /STEAM_SW -> +3.3V
Routing:
- net +3.3V: track 0.00 -> 185.3 mm, vias 0 -> 2
- net /AC_L: track 0.00 -> 100.0 mm
- net /AC_N: track 0.00 -> 75.8 mm, vias 0 -> 3
- net Net-(OC3-Pad1): track 0.00 -> 72.3 mm
- net Net-(OC2-Pad1): track 0.00 -> 38.3 mm
- net /ZC_SIGNAL: track 0.00 -> 31.8 mm
- net /ADC_IN: track 0.00 -> 24.9 mm
- net /BOILER_GPIO: track 0.00 -> 19.1 mm
- net /ADS_SCL: track 0.00 -> 17.9 mm
- net GND: track 0.00 -> 16.8 mm, vias 0 -> 6
- net Net-(J3-Pin_1): track 0.00 -> 16.3 mm
- net /PUMP_L: track 0.00 -> 16.1 mm
- net /3WAY_L: track 0.00 -> 16.0 mm
- net Net-(D1-K): track 0.00 -> 15.2 mm
- net /ADS_SDA: track 0.00 -> 15.2 mm
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- added copper zone on B.Cu, net GND
Other:
- board size 108 x 50.8 mm -> 114.3 x 63.5 mm
- board text added: "+"
- board text added: "-"
- board text added: "3v3"
- board text added: "ADC GND 3v3"
- board text added: "Axis PCB V1 github.com/Meigs2/Axis"
- board text added: "BOILER"
- board text added: "BREW"
- board text added: "DATA"
- board text added: "GND"
- board text added: "HIGH VOLTAGE!!"
- board text added: "STEAM"
- board text added: "WayWayWay"

Commit message: V1 updates
Parts:
- C1, C2: value 10nf -> 10uf
- R12, R3: value 100 -> 240
- R2, R6: value 10k -> 470
- moved R3 1.75 mm to (126.7, 72.6), turned to 180 degrees
- moved R12 1.75 mm to (121.7, 72.6), turned to 180 degrees
- moved C1 0.31 mm to (192.8, 102.4)
- moved C2 0.31 mm to (175.5, 102.4)
- moved R5 0.31 mm to (166.4, 103.8)
- moved J5 0.25 mm to (201.2, 112.0)
- moved J11 0.11 mm to (194.1, 112.0)
Routing:
- net +3.3V: track 185.3 -> 191.9 mm
- net /AC_N: track 75.8 -> 69.9 mm
- net Net-(J3-Pin_1): track 16.3 -> 11.9 mm
- net Net-(J4-Pin_1): track 12.3 -> 9.60 mm
- net /STEAM_SW: track 5.68 -> 8.03 mm
- net /BREW_SW: track 5.68 -> 8.03 mm
- net /ADS_SDA: track 15.2 -> 15.9 mm
- net Net-(C1-Pad2): track 4.76 -> 5.47 mm
- net /ADS_SCL: track 17.9 -> 18.5 mm
- net Net-(C2-Pad2): track 4.76 -> 5.33 mm
Other:
- board text added: "Axis PCB V1.0 github.com/Meigs2/Axis"
- board text removed: "Axis PCB V1 github.com/Meigs2/Axis"
