File: pcb/Axis_V1/Axis_V1.kicad_pcb (KiCad board)
At the start: 2 copper layers, 114.3 x 63.5 mm, 38 parts, among them J1 TRANSDUCER, J11 3WAY_L, J2 Screw_Terminal_01x03, J3 BREW_SW, J4 STEAM_SW, J5 AC_L, J6 AC_N, J7 BOILER_SSR, J8 Screw_Terminal_01x02, J9 PUMP_L, Q1 BC547, Q2 BT136S-600, Q3 BT136S-600, U1 Pico, U2 ADS1115IDGS, U3 MAX31855KASA

Commit message: More updates I guess
Routing:
- net +3.3V: track 191.9 -> 187.7 mm, vias 2 -> 3
Changed lines of the file:
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@@
   (via (at 130.556 113.284) (size 0.75) (drill 0.35) (layers "F.Cu" "B.Cu") (net 5))
   (via (at 131.621 113.284) (size 0.75) (drill 0.35) (layers "F.Cu" "B.Cu") (net 5))
-  (segment (start 128.778 114.3) (end 128.778 110.744) (width 0.508) (layer "F.Cu") (net 6))
-  (segment (start 128.778 110.744) (end 129.54 109.982) (width 0.508) (layer "F.Cu") (net 6))
   (segment (start 143.241 119.595) (end 135.255 111.609) (width 0.508) (layer "F.Cu") (net 6))
   (segment (start 145.034 71.374) (end 146.685 73.025) (width 0.508) (layer "F.Cu") (net 6))
@@
   (segment (start 133.08 111.996) (end 133.08 112.76) (width 0.25) (layer "F.Cu") (net 6))
   (segment (start 133.08 106.68) (end 133.08 107.696) (width 0.25) (layer "F.Cu") (net 6))
-  (segment (start 127.762 115.316) (end 128.778 114.3) (width 0.508) (layer "F.Cu") (net 6))
+  (segment (start 126.61 115.61) (end 128.12 115.61) (width 0.508) (layer "F.Cu") (net 6))
+  (segment (start 125.969 114.951) (end 125.96 114.96) (width 0.508) (layer "F.Cu") (net 6))
   (segment (start 135.255 111.609) (end 135.255 109.982) (width 0.508) (layer "F.Cu") (net 6))
-  (segment (start 125.969 115.047) (end 126.238 115.316) (width 0.508) (layer "F.Cu") (net 6))
+  (segment (start 125.969 113.369) (end 125.969 114.951) (width 0.508) (layer "F.Cu") (net 6))
   (segment (start 132.334 106.68) (end 132.842 106.68) (width 0.25) (layer "F.Cu") (net 6))
+  (segment (start 125.96 114.96) (end 126.61 115.61) (width 0.508) (layer "F.Cu") (net 6))
   (segment (start 143.51 71.374) (end 145.034 71.374) (width 0.508) (layer "F.Cu") (net 6))
-  (segment (start 125.969 113.369) (end 125.969 115.047) (width 0.508) (layer "F.Cu") (net 6))
   (segment (start 135.255 108.585) (end 133.35 106.68) (width 0.25) (layer "F.Cu") (net 6))
-  (segment (start 129.54 109.982) (end 135.255 109.982) (width 0.508) (layer "F.Cu") (net 6))
-  (segment (start 126.238 115.316) (end 127.762 115.316) (width 0.508) (layer "F.Cu") (net 6))
+  (segment (start 128.61 115.12) (end 128.61 108.585) (width 0.508) (layer "F.Cu") (net 6))
   (segment (start 132.58 107.696) (end 132.58 106.942) (width 0.25) (layer "F.Cu") (net 6))
   (segment (start 133.834 113.03) (end 135.255 111.609) (width 0.25) (layer "F.Cu") (net 6))
   (segment (start 133.35 113.03) (end 133.834 113.03) (width 0.25) (layer "F.Cu") (net 6))
+  (segment (start 128.12 115.61) (end 128.61 115.12) (width 0.508) (layer "F.Cu") (net 6))
   (segment (start 132.08 107.696) (end 132.08 106.934) (width 0.25) (layer "F.Cu") (net 6))
   (segment (start 132.842 106.68) (end 133.08 106.68) (width 0.25) (layer "F.Cu") (net 6))
   (segment (start 133.08 112.76) (end 133.35 113.03) (width 0.25) (layer "F.Cu") (net 6))
   (via (at 146.685 73.025) (size 0.75) (drill 0.35) (layers "F.Cu" "B.Cu") (net 6))
+  (via (at 128.61 108.585) (size 0.8) (drill 0.4) (layers "F.Cu" "B.Cu") (net 6))
   (via (at 135.255 108.585) (size 0.75) (drill 0.35) (layers "F.Cu" "B.Cu") (net 6))
   (segment (start 105.41 81.915) (end 105.41 80.645) (width 0.508) (layer "B.Cu") (net 6))
   (segment (start 146.685 73.025) (end 117.094 73.025) (width 0.508) (layer "B.Cu") (net 6))
-  (segment (start 135.255 108.585) (end 102.235 108.585) (width 0.508) (layer "B.Cu") (net 6))
   (segment (start 102.235 108.585) (end 97.79 104.14) (width 0.508) (layer "B.Cu") (net 6))
   (segment (start 120.221 69.898) (end 117.094 73.025) (width 0.508) (layer "B.Cu") (net 6))
   (segment (start 117.094 73.025) (end 113.03 73.025) (width 0.508) (layer "B.Cu") (net 6))
   (segment (start 120.221 66.506) (end 120.221 69.898) (width 0.508) (layer "B.Cu") (net 6))
+  (segment (start 128.61 108.585) (end 102.235 108.585) (width 0.508) (layer "B.Cu") (net 6))
   (segment (start 98.961 88.364) (end 105.41 81.915) (width 0.508) (layer "B.Cu") (net 6))
   (segment (start 92.075 103.505) (end 92.075 93.579444) (width 0.508) (layer "B.Cu") (net 6))
@@
   (segment (start 97.290444 88.364) (end 98.961 88.364) (width 0.508) (layer "B.Cu") (net 6))
   (segment (start 112.855 66.506) (end 112.855 72.85) (width 0.508) (layer "B.Cu") (net 6))
+  (segment (start 135.255 108.585) (end 128.61 108.585) (width 0.508) (layer "B.Cu") (net 6))
   (segment (start 92.71 104.14) (end 92.075 103.505) (width 0.508) (layer "B.Cu") (net 6))
   (segment (start 105.41 66.68) (end 105.41 80.645) (width 0.508) (layer "B.Cu") (net 6))

Commit message: Updates
Parts:
- removed Q1: BC547, Package_TO_SOT_THT:TO-92_Inline
- added J10: Conn_01x03, Library:1x03 Pin Header Holes, F.Cu at (163.8, 30.5)
- added J12: Conn_01x03, Library:1x03 Pin Header Holes, F.Cu at (177.8, 80.0)
- added Q4: BC847, Package_TO_SOT_SMD:SOT-23, F.Cu at (203.5, 84.8)
- H1, H2, H3, H4: footprint MountingHole:MountingHole_2.7mm_M2.5 -> MountingHole:MountingHole_4.3mm_M4
- R6: value 470 -> 20k
- moved H1 110.0 mm to (151.1, 30.5), turned to -90 degrees
- moved J3 100.1 mm to (206.9, 38.4), turned to -90 degrees
- moved J2 99.1 mm to (192.9, 28.0)
- moved H4 93.7 mm to (204.5, 30.5), turned to -90 degrees
- moved J4 91.0 mm to (206.9, 46.4), turned to -90 degrees
- moved J8 87.9 mm to (152.4, 39.4), turned to -90 degrees
- moved J7 82.4 mm to (207.0, 54.6), turned to -90 degrees
- moved H2 79.8 mm to (151.1, 121.9), turned to -90 degrees
- moved U3 76.7 mm to (161.3, 43.8), turned to 0 degrees
- moved R12 73.5 mm to (193.2, 55.9), turned to 0 degrees
- moved J1 71.5 mm to (152.4, 50.8), turned to -90 degrees
- moved U1 69.4 mm to (177.8, 52.1), turned to 0 degrees
- moved R3 67.5 mm to (193.2, 61.0), turned to 0 degrees
- moved R8 60.3 mm to (193.2, 66.0), turned to 0 degrees
- moved U2 58.3 mm to (162.2, 60.0), turned to 0 degrees
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Connections:
- U1 pad 1: unconnected-(U1-GPIO0-Pad1) -> /UART_TX
- U1 pad 2: unconnected-(U1-GPIO1-Pad2) -> /UART_RX
- U1 pad 41: unconnected-(U1-SWCLK-Pad41) -> /SWCLK
- U1 pad 42: unconnected-(U1-GND-Pad42) -> GND
- U1 pad 43: unconnected-(U1-SWDIO-Pad43) -> /SWDIO
Routing:
- net +3.3V: track 187.7 -> 0.00 mm, vias 3 -> 0
- net Net-(OC3-Pad1): track 72.3 -> 0.00 mm
- net Net-(OC2-Pad1): track 38.3 -> 0.00 mm
- net /ZC_SIGNAL: track 31.8 -> 0.00 mm
- net /ADC_IN: track 24.9 -> 0.00 mm
- net /BOILER_GPIO: track 19.1 -> 0.00 mm
- net /ADS_SCL: track 18.5 -> 0.00 mm
- net /AC_N: track 69.9 -> 52.5 mm
- net GND: track 16.6 -> 0.00 mm, vias 6 -> 0
- net /ADS_SDA: track 15.9 -> 0.00 mm
- net /MAX_SCL: track 13.3 -> 0.00 mm
- net /MAX_CS: track 12.5 -> 0.00 mm
- net /MAX_SO: track 12.0 -> 0.00 mm
- net Net-(J3-Pin_1): track 11.9 -> 0.00 mm
- net Net-(J4-Pin_1): track 9.60 -> 0.00 mm
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- removed copper zone on B.Cu, net GND
Other:
- board size 114.3 x 63.5 mm -> 63.5 x 101.6 mm
- board text removed: "+"
- board text removed: "-"
- board text removed: "3v3"
- board text removed: "ADC GND 3v3"
- board text removed: "Axis PCB V1.0 github.com/Meigs2/Axis"
- board text removed: "BOILER"
- board text removed: "BREW"
- board text removed: "DATA"
- board text removed: "GND"
- board text removed: "HIGH VOLTAGE!!"
- board text removed: "STEAM"
- board text removed: "WayWayWay"

Commit message: More and more pcb updates
Parts:
- moved U2 0.24 mm to (161.9, 60.0)
- moved C1 0.13 mm to (167.1, 112.2)
- moved C2 0.13 mm to (183.6, 112.2)
Routing:
- net +3.3V: track 0.00 -> 196.8 mm, vias 0 -> 4
- net Net-(OC3-Pad1): track 0.00 -> 49.9 mm, vias 0 -> 2
- net /MAX_SO: track 0.00 -> 33.6 mm, vias 0 -> 2
- net /MAX_SCL: track 0.00 -> 27.6 mm, vias 0 -> 2
- net Net-(OC2-Pad1): track 0.00 -> 27.6 mm, vias 0 -> 2
- net /ADC_IN: track 0.00 -> 26.5 mm
- net /MAX_CS: track 0.00 -> 25.9 mm
- net /BOILER_GPIO: track 0.00 -> 25.3 mm
- net /ZC_SIGNAL: track 0.00 -> 23.9 mm
- net Net-(J3-Pin_1): track 0.00 -> 22.6 mm
- net /ADS_SCL: track 0.00 -> 20.9 mm, vias 0 -> 1
- net Net-(J4-Pin_1): track 0.00 -> 19.7 mm
- net /ADS_SDA: track 0.00 -> 19.5 mm, vias 0 -> 1
- net /PRES_SENS: track 0.00 -> 13.2 mm
- net GND: track 0.00 -> 12.7 mm
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- added copper zone on F.Cu, net GND

Commit message: More changes
Parts:
- moved H3 32.6 mm to (181.3, 144.9)
- moved H4 32.6 mm to (181.3, 53.5)
- moved J10 32.6 mm to (140.6, 53.5)
- moved J11 32.6 mm to (138.5, 141.1)
- moved J3 32.6 mm to (183.7, 61.4)
- moved J4 32.6 mm to (183.7, 69.3)
- moved J5 32.6 mm to (181.3, 133.5)
- moved J6 32.6 mm to (181.3, 124.6)
- moved J8 32.6 mm to (129.2, 62.4)
- moved OC1 32.6 mm to (178.7, 115.7)
- moved OC3 32.6 mm to (139.4, 115.7)
- moved R5 32.6 mm to (161.0, 128.8)
- moved U1 32.6 mm to (154.6, 75.1)
- moved U2 32.6 mm to (138.7, 83.0)
- moved C1 32.6 mm to (144.0, 135.2)
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- renumbered Q4 to Q1
Routing:
- net +3.3V: track 196.8 -> 200.6 mm
Other:
- board text added: "+"
- board text added: "-"
- board text added: "3WAY_L"
- board text added: "3v3"
- board text added: "AC_L"
- board text added: "AC_N"
- board text added: "ADC"
- board text added: "BOILER_SSR"
- board text added: "BREW"
- board text added: "DATA"
- board text added: "GND"
- board text added: "PUMP_L"
- board text added: "RX"
- board text added: "STEAM"
- board text added: "TX"

Commit message: Updates again
Routing:
- net +3.3V: track 200.6 -> 201.3 mm
Other:
- board text added: "Axis PCB v1.1 github.com/Meigs2/Axis"
Changed lines of the file:
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@@
     (effects (font (size 1 1) (thickness 0.15)))
+  )
+  (gr_text "Axis PCB v1.1\ngithub.com/Meigs2/Axis" (at 123.825 100.965 270) (layer "F.SilkS")
+    (effects (font (size 1 1) (thickness 0.15)) (justify left bottom))
   )
   (gr_text "DATA" (at 136.398 73.66 270) (layer "F.SilkS")
@@
   (via (at 174.304 101.0955) (size 0.75) (drill 0.35) (layers "F.Cu" "B.Cu") (net 6))
   (via (at 147.634 104.2705) (size 0.75) (drill 0.35) (layers "F.Cu" "B.Cu") (net 6))
+  (segment (start 185.42 65.0365) (end 183.744 63.3605) (width 0.508) (layer "B.Cu") (net 6))
   (segment (start 174.304 101.0955) (end 169.224 106.1755) (width 0.508) (layer "B.Cu") (net 6))
-  (segment (start 181.474 61.0905) (end 183.744 63.3605) (width 0.508) (layer "B.Cu") (net 6))
+  (segment (start 163.509 61.0905) (end 179.8355 61.0905) (width 0.508) (layer "B.Cu") (net 6))
+  (segment (start 179.8355 61.0905) (end 182.1055 63.3605) (width 0.508) (layer "B.Cu") (net 6))
   (segment (start 170.0495 61.0905) (end 173.764 57.376) (width 0.508) (layer "B.Cu") (net 6))
   (segment (start 134.045 69.9805) (end 134.045 79.1245) (width 0.508) (layer "B.Cu") (net 6))
   (segment (start 156.845 67.7545) (end 156.845 86.36) (width 0.508) (layer "B.Cu") (net 6))
   (segment (start 156.845 86.36) (end 147.634 95.571) (width 0.508) (layer "B.Cu") (net 6))
-  (segment (start 163.509 61.0905) (end 181.474 61.0905) (width 0.508) (layer "B.Cu") (net 6))
+  (segment (start 185.42 70.485) (end 185.42 65.0365) (width 0.508) (layer "B.Cu") (net 6))
   (segment (start 163.509 61.0905) (end 156.845 67.7545) (width 0.508) (layer "B.Cu") (net 6))
-  (segment (start 185.073 64.6895) (end 183.744 63.3605) (width 0.508) (layer "B.Cu") (net 6))
   (segment (start 147.634 104.2705) (end 143.824 104.2705) (width 0.508) (layer "B.Cu") (net 6))
   (segment (start 143.824 104.2705) (end 129.219 89.6655) (width 0.508) (layer "B.Cu") (net 6))
   (segment (start 147.634 95.571) (end 147.634 104.2705) (width 0.508) (layer "B.Cu") (net 6))
   (segment (start 163.509 61.0905) (end 170.0495 61.0905) (width 0.508) (layer "B.Cu") (net 6))
-  (segment (start 185.073 70.0165) (end 185.073 64.6895) (width 0.508) (layer "B.Cu") (net 6))
+  (segment (start 183.744 71.3455) (end 184.5595 71.3455) (width 0.508) (layer "B.Cu") (net 6))
   (segment (start 169.224 106.1755) (end 167.954 106.1755) (width 0.508) (layer "B.Cu") (net 6))
   (segment (start 134.045 79.1245) (end 129.219 83.9505) (width 0.508) (layer "B.Cu") (net 6))
   (segment (start 173.764 57.376) (end 173.764 51.0155) (width 0.508) (layer "B.Cu") (net 6))
   (segment (start 129.219 89.6655) (end 129.219 83.9505) (width 0.508) (layer "B.Cu") (net 6))
-  (segment (start 183.744 71.3455) (end 185.073 70.0165) (width 0.508) (layer "B.Cu") (net 6))
+  (segment (start 182.1055 63.3605) (end 183.744 63.3605) (width 0.508) (layer "B.Cu") (net 6))
+  (segment (start 184.5595 71.3455) (end 185.42 70.485) (width 0.508) (layer "B.Cu") (net 6))
   (segment (start 165.414 73.7905) (end 163.509 73.7905) (width 0.254) (layer "F.Cu") (net 7))
   (segment (start 169.764 69.4405) (end 165.414 73.7905) (width 0.254) (layer "F.Cu") (net 7))

Commit message: v1.1 ordered, updates
Parts:
- D1: footprint Diode_SMD:D_SOD-128 -> Diode_SMD:D_SOD-123
- moved D1 1.48 mm to (172.4, 123.2)
Routing:
- net Net-(D1-K): track 8.89 -> 10.9 mm
Other:
- board text added: "WayWayWay"

Commit message: Almost messed it up.
Moved things around and make sure the rust code and schematics match up.
Parts:
- D1: value RFN1LAM6STR -> HS1MFL
- Q2, Q3: value BT136S-600 -> ACST410-8BTR
- R10: renamed from R6; value 20k -> 56k
- moved H3 78.2 mm to (198.1, 68.6), turned to 0 degrees
- moved H4 76.1 mm to (106.7, 68.6), turned to 0 degrees
- moved H2 73.8 mm to (198.1, 121.9), turned to 0 degrees
- moved J10 71.7 mm to (104.2, 80.1), turned to 90 degrees
- moved H1 71.7 mm to (106.7, 121.9), turned to 0 degrees
- moved J6 69.3 mm to (114.6, 66.1), turned to 0 degrees
- moved J3 65.3 mm to (106.7, 109.2), turned to 180 degrees
- moved J11 65.1 mm to (186.7, 68.6), turned to 90 degrees
- moved J9 63.2 mm to (194.3, 111.3), turned to 90 degrees
- moved J7 61.3 mm to (122.6, 66.1), turned to 0 degrees
- moved J8 60.7 mm to (194.3, 94.8), turned to 90 degrees
- moved J4 60.3 mm to (114.7, 120.8), turned to 0 degrees
- moved J12 56.1 mm to (177.8, 68.6), turned to 90 degrees
- moved R12 54.7 mm to (188.0, 111.3), turned to -90 degrees
- moved J2 54.3 mm to (130.8, 66.0), turned to 0 degrees
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- renumbered C2 to C1, C1 to C2, J2 to J10, J5 to J11, J6 to J12, J7 to J2, J10 to J3, J8 to J4, J12 to J5, J3 to J6, J4 to J7, J9 to J8, J11 to J9, OC3 to OC1, OC1 to OC2, OC2 to OC3, R12 to R1, R7 to R11, R10 to R12, R3 to R2, R2 to R3, R8 to R4, R1 to R5, R9 to R6, R4 to R7, R11 to R8, R5 to R9, U2 to U1, U1 to U2
Connections:
- U1 pad 10: /ADS_SDA -> /ADS_SCL
- U1 pad 9: /ADS_SCL -> /ADS_SDA
- U2 pad 14: /MAX_SO -> unconnected-(U2-GPIO10-Pad14)
- U2 pad 15: /MAX_CS -> unconnected-(U2-GPIO11-Pad15)
- U2 pad 16: /MAX_SCL -> unconnected-(U2-GPIO12-Pad16)
- U2 pad 4: unconnected-(U1-GPIO2-Pad4) -> /MAX_SCL
- U2 pad 5: unconnected-(U1-GPIO3-Pad5) -> /MAX_CS
- U2 pad 6: unconnected-(U1-GPIO4-Pad6) -> /MAX_MISO
- U3 pad 7: /MAX_SO -> /MAX_MISO
Routing:
- net /MAX_SO: track 33.6 -> 0.00 mm, vias 2 -> 0
- net /MAX_SCL: track 27.6 -> 8.91 mm, vias 2 -> 1
- net /MAX_CS: track 25.9 -> 7.40 mm, vias 0 -> 2
- net +3.3V: track 201.3 -> 188.0 mm, vias 4 -> 2
- net /PRES_SENS: track 13.2 -> 20.6 mm
- net /MAX_MISO: track 0.00 -> 6.55 mm
- net /ADS_SDA: track 19.5 -> 13.4 mm, vias 1 -> 0
- net /ADS_SCL: track 20.9 -> 18.0 mm, vias 1 -> 0
- net /NEG_THCPL: track 7.99 -> 6.10 mm
- net /POS_THCPL: track 6.41 -> 7.67 mm
- net /AC_N: track 64.6 -> 63.6 mm
Other:
- board size 63.5 x 101.6 mm -> 101.6 x 63.5 mm
