File: pcb/Axis_V1/Axis_V1.kicad_sch (KiCad schematic)
At the start: 35 parts, among them J1 Screw_Terminal_01x03, J10 BOILER_3v3, J11 3WAY_L, J2 Screw_Terminal_01x03, J3 BREW_SW, J4 STEAM_SW, J5 AC_L, J6 AC_N, J7 BOILER_GND, J9 PUMP_L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

Commit message: Updates, add Pico MCU from github
Parts:
- removed U1: Pico, MCU_RaspberryPi_and_Boards:RPi_Pico_SMD_TH, symbol Pico:Pico
- added U1: Pico, MCU_RaspberryPi_and_Boards:RPi_Pico_SMD_TH, symbol MCU_RaspberryPi_and_Boards:Pico
Connections:
- net +3.3V: now also U1.36 (3V3)
- net +5V: now also U1.40 (VBUS)
- net ADC_IN: now also U1.31 (GPIO26_ADC0)
- net GND: now also U1.13 (GND), U1.18 (GND), U1.23 (GND), U1.28 (GND), U1.3 (GND), U1.38 (GND), U1.8 (GND)
- net PIN_10: now also U1.14 (GPIO10)
- net PIN_11: now also U1.15 (GPIO11)
- net PIN_12: now also U1.16 (GPIO12)
- net PIN_13: now also U1.17 (GPIO13)
- net PIN_14: now also U1.19 (GPIO14)
- net PIN_15: now also U1.20 (GPIO15)
- net PIN_16: now also U1.21 (GPIO16)
- net PIN_17: now also U1.22 (GPIO17)
- net PIN_18: now also U1.24 (GPIO18)
- net PIN_19: now also U1.25 (GPIO19)
- net PIN_21: now also U1.27 (GPIO21)
- net PIN_22: now also U1.29 (GPIO22)

Commit message: Changes
Parts:
- OC1, OC2, OC3: footprint Package_DIP:DIP-6_W7.62mm -> Package_DIP:DIP-6_W7.62mm_LongPads
- R1: footprint Resistor_SMD:R_0805_2012Metric -> Resistor_SMD:R_1206_3216Metric
Changed lines of the file:
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@@
       (effects (font (size 1.27 1.27)))
     )
-    (property "Footprint" "Resistor_SMD:R_0805_2012Metric" (at 207.01 66.04 0)
+    (property "Footprint" "Resistor_SMD:R_1206_3216Metric" (at 207.01 66.04 0)
       (effects (font (size 1.27 1.27)) hide)
     )
@@
       (effects (font (size 1.27 1.27)))
     )
-    (property "Footprint" "Package_DIP:DIP-6_W7.62mm" (at 220.98 73.66 0)
+    (property "Footprint" "Package_DIP:DIP-6_W7.62mm_LongPads" (at 220.98 73.66 0)
       (effects (font (size 1.27 1.27) italic) (justify left) hide)
     )
@@
       (effects (font (size 1.27 1.27)))
     )
-    (property "Footprint" "Package_DIP:DIP-6_W7.62mm" (at 231.14 34.29 0)
+    (property "Footprint" "Package_DIP:DIP-6_W7.62mm_LongPads" (at 231.14 34.29 0)
       (effects (font (size 1.27 1.27) italic) (justify left) hide)
     )
@@
       (effects (font (size 1.27 1.27)))
     )
-    (property "Footprint" "Package_DIP:DIP-6_W7.62mm" (at 220.98 104.14 0)
+    (property "Footprint" "Package_DIP:DIP-6_W7.62mm_LongPads" (at 220.98 104.14 0)
       (effects (font (size 1.27 1.27) italic) (justify left) hide)
     )

Commit message: Add more stuff for pcb
Parts:
- removed C1: 100nF, Capacitor_SMD:C_0402_1005Metric, symbol Device:C_Small
- removed D1: 1N4001, Diode_THT:D_DO-41_SOD81_P10.16mm_Horizontal, symbol Diode:1N4001
- removed R6: 10k, LED_SMD:LED_2512_6332Metric, symbol Device:R_Small
- added D1: MB6S, Package_TO_SOT_SMD:TO-269AA, symbol Diode_Bridge:MB6S
- OC1: footprint Package_DIP:DIP-6_W7.62mm_LongPads -> DIP:SMDIP-6_W7.62mm
- OC2, OC3: value MOC3021M -> MOC3021S-TA1; footprint Package_DIP:DIP-6_W7.62mm_LongPads -> DIP:SMDIP-6_W7.62mm
- Q2, Q3: footprint Package_TO_SOT_THT:TO-220-3_Vertical -> Package_TO_SOT_SMD:TO-252-2
Connections:
- net +3.3V: now also OC1.6; no longer OC1.5
- net LINE: no longer OC1.2
- net PIN_10: now also U3.7 (SO); no longer U3.5 (SCK)
- net PIN_12: now also U3.5 (SCK); no longer U3.7 (SO)
- net at OC1.1: now also D1.3 (+)

Commit message: PCB Updates
Parts:
- removed C3: 100nF, Capacitor_SMD:C_0402_1005Metric, symbol Device:C_Small
- removed D1: MB6S, Package_TO_SOT_SMD:TO-269AA, symbol Diode_Bridge:MB6S
- added C1: C_Small, Resistor_SMD:R_2512_6332Metric, symbol Device:C_Small
- added D1: RFN1LAM6STR, Diode_SMD:D_SOD-128, symbol Device:D_Small
- added R6: 10k, Resistor_SMD:R_2512_6332Metric, symbol Device:R_Small
- C2: value 100nF -> C_Small; footprint Capacitor_SMD:C_0402_1005Metric -> Resistor_SMD:R_2512_6332Metric
- OC1, OC2, OC3: footprint DIP:SMDIP-6_W7.62mm -> Package_DIP:SMDIP-6_W7.62mm
- R10, R5: value 180 -> 420
- R11, R7: value 2.4k -> 420
- R2: value 1M -> 10k
- R3: value 1k -> 1M
Connections:
- net +3.3V: now also R2.2; no longer OC1.6, Q1.1 (C)
- net GND: now also Q1.3 (E), R3.1; no longer R2.1
- net LINE: now also OC2.4, OC3.4, Q2.2 (A2), Q3.2 (A2), R6.1; no longer Q2.1 (A1), Q3.1 (A1), R11.2, R7.2
- net NEUT: now also C2.1, OC1.2, C1.1, D1.2 (A)
- net PIN_16: now also OC1.5, Q1.1 (C), R2.1; no longer R3.1
- net at C2.2, R7.1: no longer R5.2
- net at R10.2: now also J11.1 (Pin_1), Q3.1 (A1); no longer R11.1
- net at Q2.3 (G): now also R5.2; no longer OC2.4
- net at R10.1: now also C1.2; no longer OC3.6
- net at OC1.1: now also D1.1 (K), R6.2
- net at OC1.4, Q1.2 (B): now also R3.2; no longer R2.2
- net at Q3.3 (G): now also R11.2; no longer OC3.4
- new net: J9.1 (Pin_1), Q2.1 (A1), R7.2
- new net: OC3.6, R11.1
- no-connect marks 22 -> 21
Other:
- moved on the sheet: J11, J9, OC1, OC3, Q2, R8, R9

Commit message: More pcb updates
Parts:
- removed R3: 1M, Resistor_SMD:R_1206_3216Metric, symbol Device:R_Small
- added H1, H2, H3, H4: MountingHole, MountingHole:MountingHole_2.7mm_M2.5, symbol Mechanical:MountingHole
- C1, C2: footprint Resistor_SMD:R_2512_6332Metric -> Capacitor_SMD:C_1206_3216Metric
- J1: value Screw_Terminal_01x03 -> TRANSDUCER
- Q2, Q3: value BT136-500 -> BT136S-600
- R1: value 200 -> 470; footprint Resistor_SMD:R_1206_3216Metric -> Resistor_SMD:R_0201_0603Metric
- R10, R7: value 420 -> 220
- R11, R5: value 420 -> 470
- R2: footprint Resistor_SMD:R_1206_3216Metric -> Resistor_SMD:R_0201_0603Metric
- R4: value 100 -> 240; footprint Resistor_SMD:R_1206_3216Metric -> Resistor_SMD:R_0201_0603Metric
- R8: value 200 -> 470
- R9: value 100 -> 240
Connections:
- net NEG_THCPL: now reaches TC1.2 (-), U3.2 (T-)
- net POS_THCPL: now reaches TC1.1 (+), U3.3 (T+)
- net PRES_SENS: now reaches J1.1 (Pin_1), U2.4 (AIN0)
- net LINE renamed AC_L
- net NEUT renamed AC_N
- net PIN_10 renamed MAX_SO
- net PIN_11 renamed MAX_CS
- net PIN_12 renamed MAX_SCL
- net PIN_13: no longer names the net of U1.17 (GPIO13)
- net PIN_13: no longer U2.2 (ALERT/RDY)
- net PIN_14 renamed ADS_SCL
- net ADS_SCL: now also U1.20 (GPIO15); no longer U1.19 (GPIO14)
- net PIN_15 renamed ADS_SDA
- net ADS_SDA: now also U1.19 (GPIO14); no longer U1.20 (GPIO15)
- net PIN_16 renamed ZC_SIGNAL
- net PIN_17 renamed PUMP_GPIO
- net PIN_18 renamed BOILER_GPIO
- net PIN_19 renamed 3WAY_GPIO
- net PIN_21 renamed STEAM_SW
- net PIN_22 renamed BREW_SW
- no-connect marks 21 -> 23
Other:
- moved on the sheet: C1, C2, D1, J1, J10, J11, J2, J3, J4, J5, J6, J7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

Commit message: We're basically there, going to get BOM together.
Parts:
- removed J10: BOILER_3v3, Library:Quick Disconnect, symbol Connector:Conn_01x01_Pin
- removed J7: BOILER_GND, Library:Quick Disconnect, symbol Connector:Conn_01x01_Pin
- removed TC1: Thermocouple_Block, TerminalBlock_RND:TerminalBlock_RND_205-00232_1x02_P5.08mm_Horizontal, symbol Device:Thermocouple_Block
- added J7: BOILER_SSR, Connector_JST:JST_PH_B2B-PH-K_1x02_P2.00mm_Vertical, symbol Connector_Generic:Conn_01x02
- added J8: Screw_Terminal_01x02, TerminalBlock_MetzConnect:TerminalBlock_MetzConnect_Type101_RT01602HBWC_1x02_P5.08mm_Horizontal, symbol Connector:Screw_Terminal_01x02
- added R12, R3: 100, Resistor_SMD:R_1206_3216Metric, symbol Device:R_Small
- C1, C2: value C_Small -> 10nf
- J2: footprint TerminalBlock_MetzConnect:TerminalBlock_MetzConnect_Type073_RT02603HBLU_1x03_P5.08mm_Horizontal -> Connector_JST:JST_PH_B3B-PH-K_1x03_P2.00mm_Vertical
- R1, R2, R4: footprint Resistor_SMD:R_0201_0603Metric -> Resistor_SMD:R_1206_3216Metric
Connections:
- net +3.3V: now also J3.2 (Pin_2), J4.2 (Pin_2); no longer J3.1 (Pin_1), J4.1 (Pin_1)
- net BOILER_GPIO: now also J7.2 (Pin_2)
- net BREW_SW: now also R12.1; no longer J3.2 (Pin_2)
- net GND: now also J7.1 (Pin_1)
- net NEG_THCPL: now also J8.1 (Pin_1)
- net POS_THCPL: now also J8.2 (Pin_2)
- net STEAM_SW: now also R3.1; no longer J4.2 (Pin_2)
- net PUMP_L: now reaches J9.1 (Pin_1), Q2.1 (A1), R7.2
- net 3WAY_L: now reaches J11.1 (Pin_1), Q3.1 (A1), R10.2
- new net: J3.1 (Pin_1), R12.2
- new net: J4.1 (Pin_1), R3.2
- no-connect marks 23 -> 24
Other:
- moved on the sheet: J2, J3, J4, Q3

Commit message: V1 updates
Parts:
- removed C1, C2: 10nf, Capacitor_SMD:C_1206_3216Metric, symbol Device:C_Small
- added C1, C2: 10uf, Capacitor_SMD:C_1206_3216Metric, symbol Device:C_Polarized_US
- R12, R3: value 100 -> 240
- R2, R6: value 10k -> 470
Connections:
- net AC_N: now also C1.1, C2.1
- net at R7.1: now also C2.2
- net at R10.1: now also C1.2
Other:
- moved on the sheet: J11, J9, R10, R7

Commit message: Updates
Parts:
- removed Q1: BC547, Package_TO_SOT_THT:TO-92_Inline, symbol Transistor_BJT:BC547
- added J10, J12: Conn_01x03, Library:1x03 Pin Header Holes, symbol Connector_Generic:Conn_01x03
- added Q4: BC847, Package_TO_SOT_SMD:SOT-23, symbol Transistor_BJT:BC847
- H1, H2, H3, H4: footprint MountingHole:MountingHole_2.7mm_M2.5 -> MountingHole:MountingHole_4.3mm_M4
- R6: value 470 -> 20k
Connections:
- net GND: now also U1.42 (GND), J10.2 (Pin_2), J12.2 (Pin_2), Q4.2 (E)
- net ZC_SIGNAL: now also Q4.3 (C)
- net UART_TX: now reaches U1.1 (GPIO0)
- net UART_TX: now also J10.3 (Pin_3)
- net UART_RX: now reaches U1.2 (GPIO1)
- net UART_RX: now also J10.1 (Pin_1)
- net SWCLK: now reaches U1.41 (SWCLK)
- net SWCLK: now also J12.1 (Pin_1)
- net SWDIO: now reaches U1.43 (SWDIO)
- net SWDIO: now also J12.3 (Pin_3)
- net at OC1.4: now also Q4.1 (B)
- no-connect marks 24 -> 19
