File: pcb/Axis_V1/Axis_V1.kicad_sch (KiCad schematic)
At the start: 40 parts, among them J1 TRANSDUCER, J10 Conn_01x03, J11 3WAY_L, J12 Conn_01x03, J2 Screw_Terminal_01x03, J3 BREW_SW, J4 STEAM_SW, J5 AC_L, J6 AC_N, J7 BOILER_SSR, J8 Screw_Terminal_01x02, J9 PUMP_L, Q2 BT136S-600, Q3 BT136S-600, Q4 BC847, U1 Pico, U2 ADS1115IDGS, U3 MAX31855KASA

Commit message: More and more pcb updates
Changed lines of the file:
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@@
+    (stroke (width 0) (type default))
+  )
+  (wire (pts (xy 242.57 66.04) (xy 242.57 67.31))
     (stroke (width 0) (type default))
   )
@@
     (stroke (width 0) (type default))
   )
+  (wire (pts (xy 242.57 99.06) (xy 242.57 100.33))
+    (stroke (width 0) (type default))
+  )
   (wire (pts (xy 139.7 172.72) (xy 130.81 172.72))
     (stroke (width 0) (type default))
@@
   )
   (wire (pts (xy 72.39 97.79) (xy 72.39 90.17))
-    (stroke (width 0) (type default))
-  )
-  (wire (pts (xy 242.57 60.96) (xy 242.57 67.31))
     (stroke (width 0) (type default))
   )
@@
     (effects (font (size 1.27 1.27)) (justify right bottom))
   )
-  (label "AC_L" (at 242.57 100.33 0) (fields_autoplaced)
+  (label "AC_L" (at 242.57 99.06 0) (fields_autoplaced)
     (effects (font (size 1.27 1.27)) (justify left bottom))
   )
@@
     (effects (font (size 1.27 1.27)) (justify right bottom))
   )
-  (label "AC_L" (at 242.57 60.96 180) (fields_autoplaced)
-    (effects (font (size 1.27 1.27)) (justify right bottom))
+  (label "AC_L" (at 242.57 66.04 0) (fields_autoplaced)
+    (effects (font (size 1.27 1.27)) (justify left bottom))
   )
   (label "NEG_THCPL" (at 100.33 172.72 0) (fields_autoplaced)

Commit message: v1.1 ordered, updates
Parts:
- D1: value RFN1LAM6STR -> HS1MFL; footprint Diode_SMD:D_SOD-128 -> Diode_SMD:D_SOD-123
- Q2, Q3: value BT136S-600 -> ACST410-8BTR
- R6: value 20k -> 56k
- renumbered Q4 to Q1
Other:
- moved on the sheet: R6
Changed lines of the file:
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@@
     (stroke (width 0) (type default))
   )
-  (wire (pts (xy 238.76 38.1) (xy 251.46 38.1))
+  (wire (pts (xy 241.3 38.1) (xy 251.46 38.1))
     (stroke (width 0) (type default))
   )
@@
     (stroke (width 0) (type default))
   )
-  (wire (pts (xy 229.87 38.1) (xy 233.68 38.1))
+  (wire (pts (xy 229.87 38.1) (xy 236.22 38.1))
     (stroke (width 0) (type default))
   )
@@
       (effects (font (size 1.27 1.27)) (justify left))
     )
-    (property "Value" "BT136S-600" (at 246.38 72.9742 0)
+    (property "Value" "ACST410-8BTR" (at 246.38 72.9742 0)
       (effects (font (size 1.27 1.27)) (justify left))
     )
@@
       (effects (font (size 1.27 1.27)) (justify left))
     )
-    (property "Value" "BT136S-600" (at 236.22 109.22 0)
+    (property "Value" "ACST410-8BTR" (at 246.38 105.41 0)
       (effects (font (size 1.27 1.27)) (justify left))
     )
@@
     )
   )
-  (symbol (lib_id "Device:R_Small") (at 236.22 38.1 270) (mirror x) (unit 1)
-    (in_bom yes) (on_board yes) (dnp no) (fields_autoplaced)
-    (property "Reference" "R6" (at 236.22 33.02 90)
-      (effects (font (size 1.27 1.27)))
-    )
-    (property "Value" "20k" (at 236.22 35.56 90)
-      (effects (font (size 1.27 1.27)))
-    )
-    (property "Footprint" "Resistor_SMD:R_2512_6332Metric" (at 236.22 38.1 0)
-      (effects (font (size 1.27 1.27)) hide)
-    )
-    (property "Datasheet" "~" (at 236.22 38.1 0)
+  (symbol (lib_id "Device:R_Small") (at 238.76 38.1 270) (mirror x) (unit 1)
+    (in_bom yes) (on_board yes) (dnp no) (fields_autoplaced)
+    (property "Reference" "R6" (at 238.76 33.02 90)
+      (effects (font (size 1.27 1.27)))
+    )
+    (property "Value" "56k" (at 238.76 35.56 90)
+      (effects (font (size 1.27 1.27)))
+    )
+    (property "Footprint" "Resistor_SMD:R_2512_6332Metric" (at 238.76 38.1 0)
+      (effects (font (size 1.27 1.27)) hide)
+    )
+    (property "Datasheet" "~" (at 238.76 38.1 0)
       (effects (font (size 1.27 1.27)) hide)
     )
@@
   (symbol (lib_id "Transistor_BJT:BC847") (at 199.39 43.18 0) (mirror y) (unit 1)
     (in_bom yes) (on_board yes) (dnp no)
-    (property "Reference" "Q4" (at 194.31 44.45 0)
+    (property "Reference" "Q1" (at 194.31 44.45 0)
       (effects (font (size 1.27 1.27)) (justify left))
     )
@@
       (project "Axis_V1"
         (path "/30841c31-0b35-46f8-9d95-4d6102b31f5d"
-          (reference "Q4") (unit 1)
+          (reference "Q1") (unit 1)
         )
       )
@@
       (effects (font (size 1.27 1.27)) (justify left))
     )
-    (property "Value" "RFN1LAM6STR" (at 232.41 41.91 90)
-      (effects (font (size 1.27 1.27)) (justify left))
-    )
-    (property "Footprint" "Diode_SMD:D_SOD-128" (at 229.87 40.64 90)
-      (effects (font (size 1.27 1.27)) hide)
-    )
+    (property "Value" "HS1MFL" (at 232.41 41.91 90)
+      (effects (font (size 1.27 1.27)) (justify left))
+    )
+    (property "Footprint" "Diode_SMD:D_SOD-123" (at 229.87 40.64 90)
+      (effects (font (size 1.27 1.27)) hide)
+    )

Commit message: Almost messed it up.
Moved things around and make sure the rust code and schematics match up.
Parts:
- renumbered C2 to C1, C1 to C2, J2 to J10, J5 to J11, J6 to J12, J7 to J2, J10 to J3, J8 to J4, J12 to J5, J3 to J6, J4 to J7, J9 to J8, J11 to J9, OC3 to OC1, OC1 to OC2, OC2 to OC3, R12 to R1, R6 to R10, R7 to R11, R10 to R12, R3 to R2, R2 to R3, R8 to R4, R1 to R5, R9 to R6, R4 to R7, R11 to R8, R5 to R9, U2 to U1, U1 to U2
Connections:
- net ADS_SCL: now also U1.10 (SCL); no longer U1.9 (SDA)
- net ADS_SDA: now also U1.9 (SDA); no longer U1.10 (SCL)
- net MAX_CS: now also U2.5 (GPIO3); no longer U2.15 (GPIO11)
- net MAX_SCL: now also U2.4 (GPIO2); no longer U2.16 (GPIO12)
- net MAX_MISO: now reaches U2.6 (GPIO4)
- net MAX_MISO: now also U3.7 (SO)
- net MAX_SO: no longer names the net of U2.14 (GPIO10)
- net MAX_SO: no longer U3.7 (SO)

Commit message: schematic updates
Parts:
- removed C1, C2: 10uf, Capacitor_SMD:C_1206_3216Metric, symbol Device:C_Polarized_US
- removed D1: HS1MFL, Diode_SMD:D_SOD-123, symbol Device:D_Small
- removed J2: BOILER_SSR, Connector_JST:JST_PH_B2B-PH-K_1x02_P2.00mm_Vertical, symbol Connector_Generic:Conn_01x02
- removed J6: BREW_SW, Connector_JST:JST_PH_B2B-PH-K_1x02_P2.00mm_Vertical, symbol Connector_Generic:Conn_01x02
- removed J7: STEAM_SW, Connector_JST:JST_PH_B2B-PH-K_1x02_P2.00mm_Vertical, symbol Connector_Generic:Conn_01x02
- removed J8: PUMP_L, Library:Quick Disconnect, symbol Connector:Conn_01x01_Pin
- removed J9: 3WAY_L, Library:Quick Disconnect, symbol Connector:Conn_01x01_Pin
- removed OC1, OC3: MOC3021S-TA1, Package_DIP:SMDIP-6_W7.62mm, symbol Relay_SolidState:MOC3021M
- removed Q2, Q3: ACST410-8BTR, Package_TO_SOT_SMD:TO-252-2, symbol Triac_Thyristor:BT136-500
- removed R1, R2, R6, R7: 240, Resistor_SMD:R_1206_3216Metric, symbol Device:R_Small
- removed R10: 56k, Resistor_SMD:R_2512_6332Metric, symbol Device:R_Small
- removed R11, R12: 220, Resistor_SMD:R_2512_6332Metric, symbol Device:R_Small
- removed R3, R4, R5: 470, Resistor_SMD:R_1206_3216Metric, symbol Device:R_Small
- removed R8, R9: 470, Resistor_SMD:R_2512_6332Metric, symbol Device:R_Small
- removed U1: ADS1115IDGS, Package_SO:TSSOP-10_3x3mm_P0.5mm, symbol Analog_ADC:ADS1115IDGS
- added C1, C2: 0.01u, symbol Device:C_Polarized_Small_US
- added C4: 0.01u, symbol Device:C_Small
- added C5: 0.1u, symbol Device:C_Polarized_Small_US
- added D1: MUR160GP, Diode_THT:D_DO-41_SOD81_P10.16mm_Horizontal, symbol Diode:1N4007
- added D2, D3: Z0107MN, Package_TO_SOT_SMD:SOT-223, symbol Triac_Thyristor:Z0107MN
- added F1: Fuse, symbol Device:Fuse
- added J10: BOILER_SSR, TerminalBlock_MetzConnect:TerminalBlock_MetzConnect_Type101_RT01602HBWC_1x02_P5.08mm_Horizontal, symbol Connector:Screw_Terminal_01x02
- added J3: BREW_SW, TerminalBlock_MetzConnect:TerminalBlock_MetzConnect_Type101_RT01602HBWC_1x02_P5.08mm_Horizontal, symbol Connector:Screw_Terminal_01x02
- added J4: PUMP_L, Library:Quick Disconnect, symbol Connector:Conn_01x01_Pin
- added J5: STEAM_SW, TerminalBlock_MetzConnect:TerminalBlock_MetzConnect_Type101_RT01602HBWC_1x02_P5.08mm_Horizontal, symbol Connector:Screw_Terminal_01x02
- added J7: 3WAY_L, Library:Quick Disconnect, symbol Connector:Conn_01x01_Pin
- added Q2: BC847, Package_TO_SOT_SMD:SOT-23, symbol Transistor_BJT:BC847
- added R1: 4.7k, symbol Device:R_Small_US
- added R10, R13, R14, R16, R6, R7: 360, symbol Device:R_Small_US
- added R11, R17: 27k, symbol Device:R_Small_US
- added R12, R9: 660, symbol Device:R_Small_US
- added R15, R5, R8: 39, symbol Device:R_Small_US
- added R18, R21: 1k, symbol Device:R_Small_US
- added R19, R22: 1.5k, symbol Device:R_Small_US
- added R2, R3: 100k, symbol Device:R_Small_US
- added R4: 0, symbol Device:R_Small_US
- added U2, U3: MOC3063M, Package_DIP:DIP-6_W7.62mm_LongPads, symbol Relay_SolidState:MOC3063M
- added U4: TPS7A0508PDBZ, Package_TO_SOT_SMD:SOT-23, symbol Regulator_Linear:TPS7A0508PDBZ
- added U6: LMV321, symbol Amplifier_Operational:LMV321
- J12: renamed from J4; value Screw_Terminal_01x02 -> THCPL
- J8: renamed from J3; value Conn_01x03 -> UART
- J9: renamed from J5; value Conn_01x03 -> DEBUG
- renumbered J11 to J1, J1 to J11, J12 to J2, J10 to J6, OC2 to OC1, U2 to U1, U3 to U5
Connections:
- net +3.3V: now also C5.1, J3.2 (Pin_2), J5.2 (Pin_2), R1.2, R13.1, R6.2; no longer J11.3 (Pin_3)
- net +5V: now also U4.3 (VI)
- net 3WAY_GPIO: now also R17.2
- net AC_L: now also D2.2 (A2), D2.4 (A4), D3.2 (A2), D3.4 (A4), F1.1, R14.2, R15.2, R4.2, R5.2, R7.2, R8.2; no longer J1.1 (Pin_1)
- net AC_N: now also C1.2, D1.2 (A)
- net BOILER_GPIO: now also J10.2 (Pin_2)
- net GND: now also OC1.4, C5.2, J10.1 (Pin_1), Q2.2 (E), R19.2, U4.1 (GND)
- net MAX_CS: now also U1.7 (GPIO5); no longer U1.5 (GPIO3)
- net PUMP_GPIO: now also R11.2
- net STEAM_SW: now also R12.2
- net ZC_SIGNAL: now also R1.1; no longer Q1.3 (C)
- net ADC_GND: now reaches U1.33 (AGND)
- net ADC_VREF: now reaches U1.35 (ADC_VREF)
- net at OC1.1: now also D1.1 (K), R2.1
- net at Q1.1 (B): now also R11.1; no longer OC1.4
- net MAX_SCL renamed MAX_SCK
- net PRES_SENS: no longer names the net of J11.1 (Pin_1)
- new net: R18.1, R19.1, U6.1 (+)
- new net: U6.3 (-), U6.4
- new net: C4.1, R15.1
- new net: C2.2, D2.1 (A1), J4.1 (Pin_1), R10.1
- new net: C4.2, D3.1 (A1), J7.1 (Pin_1), R16.1
- new net: D3.3 (G), R16.2, U3.4
- new net: D2.3 (G), R10.2, U2.4
- new net: F1.2, J1.1 (Pin_1)
- new net: J5.1 (Pin_1), R12.1
- new net: R3.2, R4.1
- new net: R2.2, R3.1
- new net: J11.3 (Pin_3), R18.2, U4.2 (VO)
- new net: R6.1, U2.1
- new net: Q1.3 (C), U2.2
- new net: R7.1, U2.6
- new net: R21.1, R22.1
- new net: Q2.1 (B), R17.1
- new net: Q2.3 (C), U3.2
- new net: C1.1, R5.1
- new net: R14.1, U3.6
- new net: R13.2, U3.1
- new net: C2.1, R8.1
- no-connect marks 19 -> 16
Other:
- note added: "R4 = Optional additional 100k for 240vac"
- note added: "UART + Debug"
- note removed: "Low Voltage Sensors/Controls"
- moved on the sheet: H1, H2, H3, H4, J1, J11, J12, J2, J6, J8, J9, OC1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

Commit message: Moreeeeeeeeeeeeee
Parts:
- removed C1, C2: 0.01u, symbol Device:C_Polarized_Small_US
- removed C4: 0.01u, symbol Device:C_Small
- removed C5: 0.1u, symbol Device:C_Polarized_Small_US
- removed D1: MUR160GP, Diode_THT:D_DO-41_SOD81_P10.16mm_Horizontal, symbol Diode:1N4007
- removed D2, D3: Z0107MN, Package_TO_SOT_SMD:SOT-223, symbol Triac_Thyristor:Z0107MN
- removed F1: Fuse, symbol Device:Fuse
- removed J1: AC_L, Library:Quick Disconnect, symbol Connector:Conn_01x01_Pin
- removed J10: BOILER_SSR, TerminalBlock_MetzConnect:TerminalBlock_MetzConnect_Type101_RT01602HBWC_1x02_P5.08mm_Horizontal, symbol Connector:Screw_Terminal_01x02
- removed J11: TRANSDUCER, TerminalBlock_MetzConnect:TerminalBlock_MetzConnect_Type073_RT02603HBLU_1x03_P5.08mm_Horizontal, symbol Connector:Screw_Terminal_01x03
- removed J12: THCPL, TerminalBlock_MetzConnect:TerminalBlock_MetzConnect_Type101_RT01602HBWC_1x02_P5.08mm_Horizontal, symbol Connector:Screw_Terminal_01x02
- removed J2: AC_N, Library:Quick Disconnect, symbol Connector:Conn_01x01_Pin
- removed J3: BREW_SW, TerminalBlock_MetzConnect:TerminalBlock_MetzConnect_Type101_RT01602HBWC_1x02_P5.08mm_Horizontal, symbol Connector:Screw_Terminal_01x02
- removed J4: PUMP_L, Library:Quick Disconnect, symbol Connector:Conn_01x01_Pin
- removed J5: STEAM_SW, TerminalBlock_MetzConnect:TerminalBlock_MetzConnect_Type101_RT01602HBWC_1x02_P5.08mm_Horizontal, symbol Connector:Screw_Terminal_01x02
- removed J6: Screw_Terminal_01x03, Connector_JST:JST_PH_B3B-PH-K_1x03_P2.00mm_Vertical, symbol Connector:Screw_Terminal_01x03
- removed J7: 3WAY_L, Library:Quick Disconnect, symbol Connector:Conn_01x01_Pin
- removed J8: UART, Library:1x03 Pin Header Holes, symbol Connector_Generic:Conn_01x03
- removed J9: DEBUG, Library:1x03 Pin Header Holes, symbol Connector_Generic:Conn_01x03
- removed OC1: 4N35, Package_DIP:SMDIP-6_W7.62mm, symbol Isolator:4N35
- removed Q1, Q2: BC847, Package_TO_SOT_SMD:SOT-23, symbol Transistor_BJT:BC847
- removed R1: 4.7k, symbol Device:R_Small_US
- removed R10, R13, R14, R16, R6, R7: 360, symbol Device:R_Small_US
- removed R11, R17: 27k, symbol Device:R_Small_US
- removed R12, R9: 660, symbol Device:R_Small_US
- removed R15, R5, R8: 39, symbol Device:R_Small_US
- removed R18, R21: 1k, symbol Device:R_Small_US
- removed R19, R22: 1.5k, symbol Device:R_Small_US
- removed R2, R3: 100k, symbol Device:R_Small_US
- removed R4: 0, symbol Device:R_Small_US
- removed U1: Pico, MCU_RaspberryPi_and_Boards:RPi_Pico_SMD_TH, symbol MCU_RaspberryPi_and_Boards:Pico
- removed U2, U3: MOC3063M, Package_DIP:DIP-6_W7.62mm_LongPads, symbol Relay_SolidState:MOC3063M
- removed U4: TPS7A0508PDBZ, Package_TO_SOT_SMD:SOT-23, symbol Regulator_Linear:TPS7A0508PDBZ
- removed U5: MAX31855KASA, Package_SO:SOIC-8_3.9x4.9mm_P1.27mm, symbol Sensor_Temperature:MAX31855KASA
- removed U6: LMV321, symbol Amplifier_Operational:LMV321
Connections:
- no-connect marks 16 -> 1
Other:
- added sheet HV Breakout (breakout.kicad_sch)
- added sheet MCU Board (mcu.kicad_sch)
- note removed: "External Boiler SSR"
- note removed: "Grouphead Thermocouple"
- note removed: "Pressure Transducer"
- note removed: "R4 = Optional additional 100k for 240vac"
- note removed: "UART + Debug"
