File: hardware/pcbs/Axis_V2/Axis_V2.kicad_pcb (KiCad board)
At the start: 2 copper layers, 0 parts

Commit message: PCB Updates
Parts:
- added C1: 0.1u, Capacitor_SMD:C_0402_1005Metric_Pad0.74x0.62mm_HandSolder, F.Cu at (118.4, 29.2)
- added C2: 0.1u, Capacitor_SMD:C_0402_1005Metric_Pad0.74x0.62mm_HandSolder, F.Cu at (83.8, 76.2)
- added C3: 0.1u, Capacitor_SMD:C_0402_1005Metric_Pad0.74x0.62mm_HandSolder, F.Cu at (120.4, 29.2)
- added C4: 0.1u, Capacitor_SMD:C_0402_1005Metric_Pad0.74x0.62mm_HandSolder, F.Cu at (127.0, 40.6)
- added C5: 0.1u, Capacitor_SMD:C_0402_1005Metric_Pad0.74x0.62mm_HandSolder, F.Cu at (127.0, 30.5)
- added J1: SWD, Connector_JST:JST_SH_BM03B-SRSS-TB_1x03-1MP_P1.00mm_Vertical, F.Cu at (84.1, 35.6)
- added J2: UART, Connector_JST:JST_SH_BM03B-SRSS-TB_1x03-1MP_P1.00mm_Vertical, F.Cu at (84.1, 27.9)
- added J3: Conn_01x02, TerminalBlock_Phoenix:TerminalBlock_Phoenix_MKDS-1,5-2-5.08_1x02_P5.08mm_Horizontal, F.Cu at (137.2, 53.3)
- added J4: Conn_01x02, TerminalBlock_Phoenix:TerminalBlock_Phoenix_MKDS-1,5-2-5.08_1x02_P5.08mm_Horizontal, F.Cu at (137.2, 68.6)
- added J5: Conn_01x04, TerminalBlock_Phoenix:TerminalBlock_Phoenix_MKDS-1,5-4-5.08_1x04_P5.08mm_Horizontal, F.Cu at (137.2, 27.9)
- added J6: Conn_01x10, TerminalBlock_RND:TerminalBlock_RND_205-00240_1x10_P5.08mm_Horizontal, F.Cu at (66.0, 73.7)
- added J7: Conn_01x08, Connector_IDC:IDC-Header_2x04_P2.54mm_Vertical, F.Cu at (97.5, 83.8)
- added R1: 1k, Resistor_SMD:R_0402_1005Metric_Pad0.72x0.64mm_HandSolder, F.Cu at (74.3, 43.9)
- added R2: 1k, Resistor_SMD:R_0402_1005Metric_Pad0.72x0.64mm_HandSolder, F.Cu at (74.3, 45.2)
- added R3: 1k, Resistor_SMD:R_0402_1005Metric_Pad0.72x0.64mm_HandSolder, F.Cu at (74.3, 42.7)
- added R4: 1k, Resistor_SMD:R_0402_1005Metric_Pad0.72x0.64mm_HandSolder, F.Cu at (116.8, 73.7)
- added R5: 1k, Resistor_SMD:R_0402_1005Metric_Pad0.72x0.64mm_HandSolder, F.Cu at (116.8, 71.1)
- added R6: 1k, Resistor_SMD:R_0402_1005Metric_Pad0.72x0.64mm_HandSolder, F.Cu at (116.8, 66.0)
- added R7: 1k, Resistor_SMD:R_0402_1005Metric_Pad0.72x0.64mm_HandSolder, F.Cu at (116.8, 63.5)
- added R8: 1k, Resistor_SMD:R_0402_1005Metric_Pad0.72x0.64mm_HandSolder, F.Cu at (116.8, 61.0)
- added R9: 1k, Resistor_SMD:R_0402_1005Metric_Pad0.72x0.64mm_HandSolder, F.Cu at (116.8, 58.4)
- added SW1: RES, Button_Switch_SMD:SW_SPST_B3U-1000P, F.Cu at (119.4, 50.8)
- added U1: Pico, MCU_RaspberryPi_and_Boards:RPi_Pico_SMD_TH, F.Cu at (101.6, 49.5)
- added U2: MAX31855EASA, Package_SO:SOIC-8_3.9x4.9mm_P1.27mm, F.Cu at (127.0, 55.9)
- added U3: MAX31855EASA, Package_SO:SOIC-8_3.9x4.9mm_P1.27mm, F.Cu at (127.0, 71.1)
- added U4: MAX6107, Package_TO_SOT_SMD:SOT-23, F.Cu at (119.4, 25.9)
- added U5: FM24CL16B, Package_SO:SOIC-8_3.9x4.9mm_P1.27mm, F.Cu at (83.8, 71.1)
- added U6: ADS1119IPWR, Package_SO:TSSOP-16_4.4x5mm_P0.65mm, F.Cu at (127.0, 35.6)
- added U7: TCA9534, Package_SO:SOIC-16W_7.5x10.3mm_P1.27mm, F.Cu at (78.1, 53.3)
Routing:
- net +3V3: track 0.00 -> 178.4 mm, vias 0 -> 5
- net /I2C0_SCL: track 0.00 -> 78.0 mm, vias 0 -> 2
- net /I2C0_SDA: track 0.00 -> 73.5 mm, vias 0 -> 5
- net /SPI0_RX: track 0.00 -> 69.2 mm, vias 0 -> 4
- net /SPI0_SCK: track 0.00 -> 66.7 mm, vias 0 -> 4
- net /SWDIO: track 0.00 -> 52.6 mm
- net /HV_IO6: track 0.00 -> 50.2 mm
- net /SPI0_CS1: track 0.00 -> 48.6 mm, vias 0 -> 3
- net /SWCLK: track 0.00 -> 46.6 mm
- net /HV_IO5: track 0.00 -> 46.3 mm
- net /SPI0_CS0: track 0.00 -> 45.8 mm, vias 0 -> 4
- net /HV_IO4: track 0.00 -> 43.2 mm, vias 0 -> 1
- net +5V: track 0.00 -> 41.8 mm, vias 0 -> 2
- net /HV_IO3: track 0.00 -> 39.2 mm
- net /HV_IO2: track 0.00 -> 36.0 mm, vias 0 -> 2
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- added copper zone on B.Cu, net GND
- added copper zone on F.Cu, net GND
Other:
- board outline added: 86.4 x 66 mm
- board text added: "GP10"
- board text added: "GP11"
- board text added: "GP12"
- board text added: "GP13"
- board text added: "GP14"
- board text added: "GP15"

Commit message: Updates
Parts:
- moved J3 3.02 mm to (136.2, 50.5)
- moved R6 3.02 mm to (115.9, 63.2), turned to 180 degrees
- moved U7 3.02 mm to (77.1, 50.5)
- moved J5 3.02 mm to (136.2, 25.1)
- moved R2 3.02 mm to (73.3, 42.4)
- moved C1 3.02 mm to (117.4, 26.4)
- moved J4 3.02 mm to (136.2, 65.7)
- moved J6 3.02 mm to (65.1, 70.8)
- moved J7 3.02 mm to (96.6, 81.0)
- moved R4 3.02 mm to (115.9, 70.8), turned to 180 degrees
- moved R5 3.02 mm to (115.9, 68.3), turned to 180 degrees
- moved R7 3.02 mm to (115.9, 60.6), turned to 180 degrees
- moved R8 3.02 mm to (115.9, 58.1), turned to 180 degrees
- moved R9 3.02 mm to (115.9, 55.6), turned to 180 degrees
- moved J2 3.02 mm to (83.1, 25.1)
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Connections:
- J7 pad 2: /HV_IO1 -> Net-(J7-Pin_2)
- J7 pad 3: /HV_IO2 -> Net-(J7-Pin_3)
- J7 pad 4: /HV_IO3 -> Net-(J7-Pin_4)
- J7 pad 5: /HV_IO4 -> Net-(J7-Pin_5)
- J7 pad 6: /HV_IO5 -> Net-(J7-Pin_6)
- J7 pad 7: /HV_IO6 -> Net-(J7-Pin_7)
- R4 pad 1: /HV_IO1 -> Net-(J7-Pin_2)
- R5 pad 1: /HV_IO2 -> Net-(J7-Pin_3)
- R6 pad 1: /HV_IO3 -> Net-(J7-Pin_4)
- R7 pad 1: /HV_IO4 -> Net-(J7-Pin_5)
- R8 pad 1: /HV_IO5 -> Net-(J7-Pin_6)
- R9 pad 1: /HV_IO6 -> Net-(J7-Pin_7)
- U1 pad 14: /SPI1_SCK_1 -> unconnected-(U1-GPIO10-Pad14)_0
- U1 pad 15: /SPI1_TX_1 -> unconnected-(U1-GPIO11-Pad15)_0
- U1 pad 16: /SPI1_RX_1 -> unconnected-(U1-GPIO12-Pad16)_0
- U1 pad 17: /SPI1_CS0_1 -> unconnected-(U1-GPIO13-Pad17)_0
- U1 pad 5: /SPI0_TX -> unconnected-(U1-GPIO3-Pad5)
Routing:
- net /HV_IO6: track 50.2 -> 5.75 mm
- net Net-(J7-Pin_7): track 0.00 -> 44.4 mm
- net /HV_IO5: track 46.3 -> 5.75 mm
- net Net-(J7-Pin_6): track 0.00 -> 40.5 mm
- net /HV_IO4: track 43.2 -> 5.75 mm, vias 1 -> 0
- net Net-(J7-Pin_5): track 0.00 -> 37.5 mm, vias 0 -> 1
- net Net-(J7-Pin_4): track 0.00 -> 33.5 mm
- net /HV_IO3: track 39.2 -> 5.75 mm
- net /HV_IO2: track 36.0 -> 5.75 mm, vias 2 -> 0
- net Net-(J7-Pin_3): track 0.00 -> 30.3 mm, vias 0 -> 2
- net Net-(J7-Pin_2): track 0.00 -> 23.1 mm
- net /HV_IO1: track 28.8 -> 5.75 mm
- net /4.5V_VREF: track 16.1 -> 17.2 mm
- net +5V: track 41.8 -> 41.2 mm
- net /SPI0_RX: track 69.2 -> 68.7 mm
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