File: hardware/pcbs/Axis_V2_HV/Axis_V2_HV.kicad_sch (KiCad schematic)
At the start: 22 parts, among them J1 AC_L, J2 AC_N, Q1 BC847, Q2 BC847, U1 AQH3213, U2 AQH3213

Commit message: More changes, wow! Who would have thought?
Parts:
- removed J1: AC_L, Footprints:Quick Disconnect, symbol Connector:Conn_01x01_Pin
- removed J2: AC_N, Footprints:Quick Disconnect, symbol Connector:Conn_01x01_Pin
- added C3: 10nf, Capacitor_SMD:C_1206_3216Metric, symbol Device:C_Small
- added F2, F3: Fuse (1A), Fuse:Fuseholder_Cylinder-5x20mm_Schurter_0031_8201_Horizontal_Open, symbol Device:Fuse_Small
- added J1: Screw_Terminal_01x03, symbol Connector:Screw_Terminal_01x03
- added J2, J4: 3WAY, symbol Connector:Screw_Terminal_01x02
- added J5: PUMP, symbol Connector:Screw_Terminal_01x02
- added K1: G2RL-1-E, Relay_THT:Relay_SPDT_Omron_G2RL-1-E, symbol Relay:G2RL-1-E
- added U3: SZNUD3160, symbol Project_Library:SZNUD3160
- F1: value Fuse -> Fuse (15A)
- RV1: value 10D471K -> Varistor
Connections:
- net 3WAY_L: now also J2.1 (Pin_1), J4.1 (Pin_1), J5.1 (Pin_1)
- net AC_L: now also RV1.1, F2.2, F3.2; no longer R6.1, R7.1, R8.1, R9.1, RV1.2, U1.8, U2.8
- net AC_N: now also RV1.2, J1.2 (Pin_2), J2.2 (Pin_2), J4.2 (Pin_2), J5.2 (Pin_2); no longer RV1.1
- net GND: now also U3.2 (GND)
- net at D1.1 (K), OC1.1, R9.2: no longer R10.2, R8.2
- net AC_HOT: now reaches F1.2
- net AC_HOT: now also J1.1 (Pin_1), K1.14
- new net: R10.2, R8.1
- new net: F3.1, R7.1, U2.8
- new net: F2.1, R6.1, U1.8
- new net: R8.2, R9.1
- new net: C3.2, K1.A2, U3.3 (OUT)
- new net +5V: C3.1, K1.A1
- new net AC_SWITCHED: J1.3 (Pin_3), K1.11
- new net PWR_SW: U3.1 (IN)
- no-connect marks 3 -> 4
Other:
- note added: "120/240v compatable, one resistor with 0r"
- moved on the sheet: C1, C2, D1, F1, OC1, Q1, Q2, R1, R2, R3, R4, R5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

Commit message: More updates and changes
Parts:
- removed J2: 3WAY, symbol Connector:Screw_Terminal_01x02
- added J2: Conn_01x08, Connector_IDC:IDC-Header_2x04_P2.54mm_Vertical, symbol Connector_Generic:Conn_01x08
- F1: value Fuse (15A) -> Fuse (15A, slow)
- F2, F3: value Fuse (1A) -> Fuse (1A, fast)
- R4, R5: value 165 -> 160
Connections:
- net +3V3: now also J2.2 (Pin_2)
- net +5V: now also J2.1 (Pin_1)
- net 3WAY_L: no longer J5.1 (Pin_1)
- net AC_L: now also RV1.2; no longer RV1.1
- net AC_N: now also RV1.1; no longer RV1.2
- net GND: now also J2.8 (Pin_8)
- net PUMP_L: now also J5.1 (Pin_1)
- new net HV_IO1: J2.3 (Pin_3)
- new net HV_IO2: J2.4 (Pin_4)
- new net HV_IO3: J2.5 (Pin_5)
- new net HV_IO4: J2.6 (Pin_6)
- new net HV_IO5: J2.7 (Pin_7)
Other:
- moved on the sheet: C1, C2, C3, D1, F1, F2, F3, J1, J4, J5, K1, OC1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

Commit message: Add "V3"
Parts:
- removed D1: 1N4007, Diode_THT:D_DO-41_SOD81_P10.16mm_Horizontal, symbol Device:D_Small
- added C5: 1n, Capacitor_SMD:C_1206_3216Metric, symbol Device:C_Small
- added C6: 10u, Capacitor_SMD:C_1206_3216Metric, symbol Device:C_Small
- added D1: MB6S, Package_TO_SOT_SMD:TO-269AA, symbol Diode_Bridge:MB6S
- added D2: ?, Diode_SMD:D_1206_3216Metric, symbol Device:D
- added J3: 3WAY, TerminalBlock_Phoenix:TerminalBlock_Phoenix_MKDS-1,5-2-5.08_1x02_P5.08mm_Horizontal, symbol Connector:Screw_Terminal_01x02
- added PS1: IRM-10-5, Converter_ACDC:Converter_ACDC_MeanWell_IRM-10-xx_THT, symbol Converter_ACDC:IRM-10-5
- added Q3: MMBT3904, Package_TO_SOT_SMD:SOT-23, symbol Transistor_BJT:MMBT3904
- added R11: 1k, LED_SMD:LED_1206_3216Metric, symbol Device:R_Small
- added R12, R13, R14: 1k, Resistor_SMD:R_0402_1005Metric, symbol Device:R_Small
- added U4: PCA9536DP, Package_SO:TSSOP-8_3x3mm_P0.65mm, symbol Interface_Expansion:PCA9536DP
- C1, C2: value 10nf -> 0.1u; footprint Capacitor_SMD:C_1206_3216Metric -> (none)
- F2, F3: value Fuse (1A, fast) -> Fuse (1A, Slow)
- J1: footprint (none) -> TerminalBlock_Phoenix:TerminalBlock_Phoenix_MKDS-1,5-3-5.08_1x03_P5.08mm_Horizontal
- J4, J5: footprint (none) -> TerminalBlock_Phoenix:TerminalBlock_Phoenix_MKDS-1,5-2-5.08_1x02_P5.08mm_Horizontal
- R1, R2, R3: value 4.7k -> 1k; footprint Resistor_SMD:R_0603_1608Metric_Pad0.98x0.95mm_HandSolder -> Resistor_SMD:R_0402_1005Metric
- R10: value 100k -> 22k; footprint (none) -> Resistor_SMD:R_1206_3216Metric
- R4, R5: value 160 -> 162
- R6, R7: value 39 -> 47
- R8, R9: value 100k -> 220k
- RV1: value Varistor -> MOV-10D471K; footprint (none) -> Varistor:RV_Disc_D12mm_W7.5mm_P7.5mm
- U3: footprint (none) -> Package_TO_SOT_SMD:SOT-23
Connections:
- net HV_IO1 is gone; now on net PUMP_IN: J2.3 (Pin_3)
- net HV_IO5 is gone; now on net 3WAY_IN: J2.7 (Pin_7)
- net +3V3: now also R12.2, U4.8 (VDD); no longer R3.1
- net AC_N: now also R8.2; no longer OC1.2
- net GND: now also J3.2 (Pin_2), U4.4 (VSS)
- net PWR_SW: now also U4.1 (IO0)
- net ~{ZC_SIG}: now also R14.1; no longer R3.2
- net at R10.2: now also D1.4 (-), D2.1 (K), Q3.1 (B); no longer R8.1
- net at OC1.1: now also R11.2; no longer R9.2
- net at R9.1: now also C5.1, D1.1; no longer R8.2
- net AC_HOT renamed AC_POS
- net AC_L renamed AC_P
- net AC_P: now also R9.2; no longer R10.1
- net HV_IO2 renamed ZC_SIG
- net HV_IO3 renamed HV_SDA
- net HV_SDA: now also U4.7 (SDA)
- net HV_IO4 renamed HV_SCL
- net HV_SCL: now also U4.6 (SCL)
- new net: C6.2, D2.2 (A), Q3.2 (E)
- new net: R12.1, R3.2
- new net: OC1.2, Q3.3 (C)
- new net: C6.1, D1.3 (+), R10.1, R11.1
- new net: R13.2, R14.2
- new net: R13.1, R3.1
- new net: C5.2, D1.2, R8.1
- new net SSR: J3.1 (Pin_1), U4.2 (IO1)
- no-connect marks 4 -> 6
Other:
- note added: "All components left of 220k R's should be 16v rated, should typically see ~5v max"
- note added: "I have a lot of 1k resistors, replace with 3.3k in final PCB."
- note added: "In the future, could use an external 5v power supply like the IRM-10-5"
- note added: "Pull-up resistors for I2C lines not required, they are on the control board."
- note added: "ZC Mains Detector (Ctrl-click for link)"
- note removed: "120/240v compatable, one resistor with 0r"
- moved on the sheet: C1, C2, C3, F2, F3, J1, J2, J4, J5, K1, Q1, Q2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

Commit message: Updates to the HV pcb
Parts:
- removed D2: ?, Diode_SMD:D_1206_3216Metric, symbol Device:D
- added C4: 0.1u, Capacitor_THT:C_Rect_L13.0mm_W6.0mm_P10.00mm_FKS3_FKP3_MKS4, symbol Device:C_Small
- added D2: 1N4148W, Diode_SMD:D_SOD-123, symbol Diode:1N4148W
- added R15: 220, Resistor_THT:R_Axial_DIN0207_L6.3mm_D2.5mm_P10.16mm_Horizontal, symbol Device:R_Small
- added RV2, RV3: MOV-10D471K, Varistor:RV_Disc_D12mm_W7.5mm_P7.5mm, symbol Device:Varistor
- C1, C2: footprint (none) -> Capacitor_THT:C_Rect_L13.0mm_W6.0mm_P10.00mm_FKS3_FKP3_MKS4
- R4, R5: footprint Resistor_SMD:R_0603_1608Metric_Pad0.98x0.95mm_HandSolder -> Resistor_SMD:R_0603_1608Metric
- R6, R7: value 47 -> 220; footprint (none) -> Resistor_THT:R_Axial_DIN0207_L6.3mm_D2.5mm_P10.16mm_Horizontal
- R8, R9: footprint (none) -> Resistor_THT:R_Axial_DIN0207_L6.3mm_D2.5mm_P10.16mm_Horizontal
Connections:
- net 3WAY_L: no longer C2.2, U2.6
- net AC_N: no longer RV1.1
- net AC_P: no longer RV1.2
- net AC_POS: now also R7.1, RV3.2
- net AC_SWITCHED: now also C2.2, RV3.1
- net PUMP_L: now also RV1.1, U2.6, C4.2, RV2.1
- net at D1.4 (-), Q3.1 (B), R10.2: now also D2.1 (K)
- net at C6.2, Q3.2 (E): now also D2.2 (A)
- net at F3.1, U2.8: now also R15.1, RV2.2; no longer R7.1
- net at F2.1, R6.1, U1.8: now also RV1.2
- new net: C4.1, R15.2
Other:
- note added: "1/4W"
- note added: "Snubber Caps are X2 Rated B32921C3104M289"
- moved on the sheet: F2, R10, R14

Commit message: Oops haha changes
Other:
- note added: "Fuse Holders: SCHURTER 0031.8201"
Changed lines of the file:
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@@
+		)
+	)
+	(text "Fuse Holders:\n\n	\nSCHURTER 0031.8201"
+		(exclude_from_sim no)
+		(at 254.254 108.204 0)
+		(effects
+			(font
+				(size 1.27 1.27)
+			)
 		)
 	)

Commit message: Is anyone listening anymore?
Parts:
- removed C2: 0.1u, Capacitor_THT:C_Rect_L13.0mm_W6.0mm_P10.00mm_FKS3_FKP3_MKS4, symbol Device:C_Small
- removed C3: 10nf, Capacitor_SMD:C_1206_3216Metric, symbol Device:C_Small
- removed J1: Screw_Terminal_01x03, TerminalBlock_Phoenix:TerminalBlock_Phoenix_MKDS-1,5-3-5.08_1x03_P5.08mm_Horizontal, symbol Connector:Screw_Terminal_01x03
- removed K1: G2RL-1-E, Relay_THT:Relay_SPDT_Omron_G2RL-1-E, symbol Relay:G2RL-1-E
- removed R7: 220, Resistor_THT:R_Axial_DIN0207_L6.3mm_D2.5mm_P10.16mm_Horizontal, symbol Device:R_Small
- removed RV3: MOV-10D471K, Varistor:RV_Disc_D12mm_W7.5mm_P7.5mm, symbol Device:Varistor
- removed U3: SZNUD3160, Package_TO_SOT_SMD:SOT-23, symbol Project_Library:SZNUD3160
- added C7: 0.1u, Capacitor_SMD:C_0402_1005Metric, symbol Device:C_Small
- added H1, H2, H3, H4: MountingHole, MountingHole:MountingHole_2.7mm_M2.5, symbol Mechanical:MountingHole
- added J2: AC, TerminalBlock_Phoenix:TerminalBlock_Phoenix_MKDS-1,5-2-5.08_1x02_P5.08mm_Horizontal, symbol Connector:Screw_Terminal_01x02
- added J6: PWR, TerminalBlock_Phoenix:TerminalBlock_Phoenix_MKDS-1,5-2-5.08_1x02_P5.08mm_Horizontal, symbol Connector:Screw_Terminal_01x02
- F1: value Fuse (15A, slow) -> Fuse (3A, slow)
- J5: renamed from J3; value 3WAY -> SSR
- renumbered C6 to C1, C5 to C2, C1 to C3, J2 to J1, J5 to J3, Q3 to Q1, Q1 to Q2, Q2 to Q3, R12 to R1, R6 to R10, R1 to R11, R5 to R12, R15 to R13, R2 to R14, R3 to R2, R13 to R3, R14 to R4, R11 to R5, R9 to R6, R10 to R7, R4 to R9, U4 to U2, U2 to U3
Connections:
- net +3V3: now also C7.1
- net 3WAY_L: now also C4.2, RV2.1, U3.6
- net AC_POS: now also J2.1 (Pin_1)
- net GND: now also C7.2, J6.2 (Pin_2)
- net PUMP_L: no longer C4.2, RV2.1, U3.6
- net PWR_SW: now also J6.1 (Pin_1)
- net AC_N renamed AC_NEG
- net AC_NEG: now also J2.2 (Pin_2)
- no-connect marks 6 -> 5
Other:
- moved on the sheet: C1, C2, C3, C4, D1, D2, F1, F2, F3, OC1, Q1, Q2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

Commit message: Yuuuuuuuuuuuuuuuuuup, nobody's here
Parts:
- R5: footprint LED_SMD:LED_1206_3216Metric -> Resistor_SMD:R_1206_3216Metric
Connections:
- net ZC_SIG is gone; now on net ~{ZC_SIG}: J1.4 (Pin_4)
Changed lines of the file:
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@@
+		)
+	)
+	(label "~{ZC_SIG}"
+		(at 66.04 43.18 180)
+		(fields_autoplaced yes)
+		(effects
+			(font
+				(size 1.27 1.27)
+			)
+			(justify right bottom)
 		)
 	)
@@
 	(label "AC_POS"
 		(at 264.16 33.02 180)
-		(fields_autoplaced yes)
-		(effects
-			(font
-				(size 1.27 1.27)
-			)
-			(justify right bottom)
-		)
-	)
-	(label "ZC_SIG"
-		(at 66.04 43.18 180)
 		(fields_autoplaced yes)
 		(effects
@@
 			)
 		)
-		(property "Footprint" "LED_SMD:LED_1206_3216Metric"
+		(property "Footprint" "Resistor_SMD:R_1206_3216Metric"
 			(at 160.02 33.02 0)
 			(effects

Commit message: Ok I'm about to order the HV pcb and parts somebody stop me
Parts:
- F1: value Fuse (3A, slow) -> Fuse (1.5A, slow)
- F2, F3: value Fuse (1A, Slow) -> Fuse (0.5A, Slow?)
Other:
- moved on the sheet: F1, H1, H2, H3, H4, J5, J6
