File: hardware/pcbs/Axis_MCU_V3/Axis_MCU_V3.kicad_pcb (KiCad board)
At the start: 4 copper layers, 90 x 60 mm, 51 parts, among them J1 SWD, J10 HV_IDC, J2 GPIO, J3 Conn_01x04, J4 UART, J5 Conn_01x02, J7 EXT_SPI, J8 EXT_I2C, J9 GPIO, SW1 RES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

Commit message: Rev 3 Update or something
Parts:
- U5: value PCA9544APW -> PCA9544APWR
- moved J1 57.1 mm to (80.0, 33.4), turned to 180 degrees
- moved J4 6.60 mm to (72.0, 33.4)
- moved R5 2.14 mm to (119.4, 76.8), turned to 180 degrees
- moved R4 1.86 mm to (117.4, 76.8), turned to 0 degrees
Connections:
- R4 pad 2: /I2C1_SDA -> /I2C1_SCL
- R5 pad 2: /I2C1_SCL -> /I2C1_SDA
- U1 pad 26: /I2C1_SDA -> /HV_IO1
- U1 pad 27: /I2C1_SCL -> /ZC_SIG
- U1 pad 31: /HV_IO1 -> /I2C1_SDA
- U1 pad 32: /ZC_SIG -> /I2C1_SCL
Routing:
- net +3V3: track 52.2 -> 241.1 mm
- net /SWDIO: track 4.66 -> 107.7 mm
- net /SWCLK: track 4.66 -> 95.4 mm
- net /I2C1_SCL: track 45.4 -> 74.4 mm
- net /HV_IO1: track 34.0 -> 53.0 mm, vias 0 -> 2
- net /I2C1_SDA: track 49.4 -> 66.7 mm
- net /ZC_SIG: track 30.3 -> 45.4 mm
- net /UART_RX: track 16.8 -> 21.1 mm
- net /UART_TX: track 21.6 -> 25.7 mm
- net GND: track 44.8 -> 41.5 mm, vias 44 -> 45
- net /HV_SCL: track 54.5 -> 55.4 mm
- net /I2C0_SDA: track 30.5 -> 31.3 mm
- net /HV_SDA: track 50.6 -> 51.4 mm
- net /SPI1_RX: track 8.98 -> 9.76 mm
- net /~{SPI1_CS0}: track 8.90 -> 9.61 mm
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Other:
- board text added: "Axis PCB V2 Rev. 2 Meigs2"
- board text removed: "Axis PCB V2 Rev. 1 Meigs2"
