File: hardware/pcbs/Axis_MCU_V3/Axis_MCU_V3.kicad_sch (KiCad schematic)
At the start: 54 parts, among them J1 SWD, J10 HV_IDC, J2 GPIO, J3 Conn_01x04, J4 UART, J5 Conn_01x02, J6 Conn_01x02, J7 EXT_SPI, J8 EXT_I2C, J9 GPIO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

Commit message: Add "V3"
Parts:
- removed C6: 0.1u, Capacitor_SMD:C_0603_1608Metric_Pad1.08x0.95mm_HandSolder, symbol Device:C_Small
- removed J6: Conn_01x02, TerminalBlock_Phoenix:TerminalBlock_Phoenix_MKDS-1,5-2-5.08_1x02_P5.08mm_Horizontal, symbol Connector_Generic:Conn_01x02
- removed U5: PCA9544AD, Package_SO:SOIC-20W_7.5x12.8mm_P1.27mm, symbol Interface_Expansion:PCA9544AD
- removed U6: MAX31855EASA, Package_SO:SOIC-8_3.9x4.9mm_P1.27mm, symbol Sensor_Temperature:MAX31855EASA
- added R15: 1k, Resistor_SMD:R_0402_1005Metric, symbol Device:R_Small
- added U5: PCA9544APWR, Package_SO:TSSOP-20_4.4x6.5mm_P0.65mm, symbol Interface_Expansion:PCA9544APW
- C1, C10, C2, C3, C4, C5, C7, C8, C9: footprint Capacitor_SMD:C_0603_1608Metric_Pad1.08x0.95mm_HandSolder -> Capacitor_SMD:C_0402_1005Metric
- R1, R10, R11, R12, R13, R14, R16, R17, R18, R2, R3, R4, R5, R6, R7, R8, R9: footprint Resistor_SMD:R_0603_1608Metric_Pad0.98x0.95mm_HandSolder -> Resistor_SMD:R_0402_1005Metric
- U1: footprint MCU_RaspberryPi_and_Boards:RPi_Pico_SMD_TH -> MCU_RaspberryPi_and_Boards:RPi_Pico_SMD_TH_No_Silkscreen
Connections:
- net +3V3: now also R15.1, U5.20 (VDD)
- net ADS_SCL: now also U5.9 (SC1)
- net ADS_SDA: now also U5.8 (SD1)
- net EXT_SCL: now also U5.13 (SC2)
- net EXT_SDA: now also U5.12 (SD2)
- net GND: now also U5.1 (A0), U5.10 (VSS), U5.2 (A1), U5.3 (A2)
- net HV_SCL: now also U5.16 (SC3)
- net HV_SDA: now also U5.15 (SD3)
- net I2C1_SCL: now also U5.18 (SCL)
- net I2C1_SDA: now also U5.19 (SDA)
- net TIMER_SCL: now also U5.6 (SC0)
- net TIMER_SDA: now also U5.5 (SD0)
- net ~{ADS_RDY}: now also U5.7 (~{INT1})
- net ~{EXT_INT}: now also U5.11 (~{INT2})
- net ~{MUX_INT}: now also U5.17 (~{INT})
- net ~{TIMER_INT}: now also U5.4 (~{INT0})
- new net ~{INT_3}: R15.2, U5.14 (~{INT3})
- no-connect marks 12 -> 11
Other:
- note added: "SM03B-SRSS-TB"
- moved on the sheet: BT1, C10, H1, H2, H3, H4, U9

Commit message: Rev 3 Update or something
Connections:
- net HV_IO1: now also U1.26 (GPIO20); no longer U1.31 (GPIO26_ADC0)
- net I2C1_SCL: now also R4.2, U1.32 (GPIO27_ADC1); no longer R5.2, U1.27 (GPIO21)
- net I2C1_SDA: now also R5.2, U1.31 (GPIO26_ADC0); no longer R4.2, U1.26 (GPIO20)
- net ZC_SIG: now also U1.27 (GPIO21); no longer U1.32 (GPIO27_ADC1)
Changed lines of the file:
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@@
 	)
 	(junction
+		(at 101.6 102.87)
+		(diameter 0)
+		(color 0 0 0 0)
+	)
+	(junction
 		(at 255.27 60.96)
 		(diameter 0)
@@
 	)
 	(junction
-		(at 95.25 95.25)
-		(diameter 0)
-		(color 0 0 0 0)
-	)
-	(junction
 		(at 243.84 143.51)
 		(diameter 0)
@@
 	)
 	(junction
-		(at 101.6 97.79)
+		(at 95.25 105.41)
 		(diameter 0)
 		(color 0 0 0 0)
@@
 	(wire
 		(pts
+			(xy 74.93 105.41) (xy 95.25 105.41)
+		)
+		(stroke
+			(width 0)
+			(type default)
+		)
+	)
+	(wire
+		(pts
 			(xy 255.27 60.96) (xy 255.27 64.77)
 		)
@@
 	(wire
 		(pts
-			(xy 74.93 95.25) (xy 95.25 95.25)
-		)
-		(stroke
-			(width 0)
-			(type default)
-		)
-	)
-	(wire
-		(pts
 			(xy 312.42 142.24) (xy 312.42 140.97)
 		)
@@
 	(wire
 		(pts
+			(xy 101.6 102.87) (xy 123.19 102.87)
+		)
+		(stroke
+			(width 0)
+			(type default)
+		)
+	)
+	(wire
+		(pts
 			(xy 246.38 34.29) (xy 246.38 35.56)
 		)
@@
 	(wire
 		(pts
-			(xy 101.6 97.79) (xy 101.6 93.98)
-		)
-		(stroke
-			(width 0)
-			(type default)
-		)
-	)
-	(wire
-		(pts
 			(xy 95.25 88.9) (xy 95.25 87.63)
 		)
@@
 	(wire
 		(pts
-			(xy 74.93 107.95) (xy 88.9 107.95)
+			(xy 74.93 107.95) (xy 123.19 107.95)
 		)
 		(stroke
@@
 	(wire
 		(pts
-			(xy 74.93 97.79) (xy 101.6 97.79)
-		)
-		(stroke
-			(width 0)
-			(type default)
-		)
-	)
-	(wire
-		(pts
 			(xy 101.6 87.63) (xy 101.6 88.9)
 		)
@@
 	(wire
 		(pts
-			(xy 95.25 95.25) (xy 95.25 93.98)
-		)
-		(stroke
-			(width 0)
-			(type default)
-		)
-	)
-	(wire
-		(pts
 			(xy 273.05 71.12) (xy 273.05 72.39)
 		)
@@
 	(wire
 		(pts
-			(xy 74.93 105.41) (xy 88.9 105.41)
-		)
-		(stroke
-			(width 0)
-			(type default)
-		)
-	)
-	(wire
-		(pts
 			(xy 107.95 138.43) (xy 107.95 139.7)
 		)
@@
 	(wire
 		(pts
+			(xy 95.25 105.41) (xy 123.19 105.41)
+		)
+		(stroke
+			(width 0)
+			(type default)
+		)
+	)
+	(wire
+		(pts
 			(xy 140.97 147.32) (xy 140.97 149.86)
 		)
@@
 	(wire
 		(pts
-			(xy 95.25 95.25) (xy 123.19 95.25)
+			(xy 74.93 95.25) (xy 88.9 95.25)
 		)
 		(stroke
@@
 	(wire
 		(pts
+			(xy 101.6 93.98) (xy 101.6 102.87)
+		)
+		(stroke
+			(width 0)
+			(type default)
+		)
+	)
+	(wire
+		(pts
 			(xy 186.69 43.18) (xy 205.74 43.18)
 		)
@@
 	(wire
 		(pts
+			(xy 74.93 102.87) (xy 101.6 102.87)
+		)
+		(stroke
+			(width 0)
+			(type default)
+		)
+	)
+	(wire
+		(pts
 			(xy 317.5 167.64) (xy 317.5 168.91)
 		)
@@
 	(wire
 		(pts
-			(xy 101.6 97.79) (xy 123.19 97.79)
-		)
-		(stroke
-			(width 0)
-			(type default)
-		)
-	)
-	(wire
-		(pts
 			(xy 299.72 177.8) (xy 317.5 177.8)
 		)
@@
 	(wire
 		(pts
+			(xy 95.25 93.98) (xy 95.25 105.41)
+		)
+		(stroke
+			(width 0)
+			(type default)
+		)
+	)
+	(wire
+		(pts
 			(xy 101.6 62.23) (xy 107.95 62.23)
 		)
@@
 	(wire
 		(pts
-			(xy 74.93 102.87) (xy 88.9 102.87)
+			(xy 74.93 97.79) (xy 88.9 97.79)
 		)
 		(stroke
@@
 		)
 	)
+	(label "HV_IO2"
+		(at 123.19 107.95 180)
+		(fields_autoplaced yes)
+		(effects
+			(font
+				(size 1.27 1.27)
+			)
+			(justify right bottom)
+		)
+	)
 	(label "IO_2"
 		(at 191.77 38.1 180)
@@
 		)
 	)
-	(label "ZC_SIG"
-		(at 88.9 105.41 180)
-		(fields_autoplaced yes)
-		(effects
-			(font
-				(size 1.27 1.27)
-			)
-			(justify right bottom)
-		)
-	)
 	(label "SWCLK"
 		(at 27.94 39.37 0)
@@
 		)
 	)
-	(label "HV_IO2"
-		(at 88.9 107.95 180)
-		(fields_autoplaced yes)
-		(effects
-			(font
-				(size 1.27 1.27)
-			)
-			(justify right bottom)
-		)
-	)
 	(label "UART_RX"
 		(at 102.87 46.99 0)
@@
 	)
 	(label "I2C1_SDA"
-		(at 123.19 95.25 180)
+		(at 123.19 102.87 180)
 		(fields_autoplaced yes)
 		(effects
@@
 		)
 	)
-	(label "HV_IO1"
-		(at 88.9 102.87 180)
-		(fields_autoplaced yes)
-		(effects
-			(font
-				(size 1.27 1.27)
-			)
-			(justify right bottom)
-		)
-	)
 	(label "TIMER_SDA"
 		(at 299.72 142.24 0)
@@
 		)
 	)
-	(label "I2C1_SCL"
-		(at 123.19 97.79 180)
+	(label "I2C0_SCL"
+		(at 31.75 148.59 0)
 		(fields_autoplaced yes)
 		(effects
@@
 				(size 1.27 1.27)
 			)
-			(justify right bottom)
+			(justify left bottom)
 		)
 	)
-	(label "I2C0_SCL"
-		(at 31.75 148.59 0)
+	(label "I2C1_SCL"
+		(at 123.19 105.41 180)
 		(fields_autoplaced yes)
 		(effects
@@
 				(size 1.27 1.27)
 			)
-			(justify left bottom)
+			(justify right bottom)
 		)
 	)
@@
 		)
 	)
+	(label "HV_IO1"
+		(at 88.9 95.25 180)
+		(fields_autoplaced yes)
+		(effects
+			(font
+				(size 1.27 1.27)
+			)
+			(justify right bottom)
+		)
+	)
 	(label "EXT_SDA"
 		(at 299.72 175.26 0)
@@
 		)
 	)
+	(label "ZC_SIG"
+		(at 88.9 97.79 180)
+		(fields_autoplaced yes)
+		(effects
+			(font
+				(size 1.27 1.27)
+			)
+			(justify right bottom)
+		)
+	)
 	(label "GPIO3"
 		(at 88.9 46.99 180)
@@
 	)
 	(symbol
-		(lib_name "+3V3_1")
-		(lib_id "power:+3V3")
-		(at 95.25 86.36 0)
-		(unit 1)
-		(exclude_from_sim no)
-		(in_bom yes)
-		(on_board yes)
-		(dnp no)
-		(fields_autoplaced yes)
-		(property "Reference" "#PWR027"
-			(at 95.25 90.17 0)
-			(effects
-				(font
-					(size 1.27 1.27)
-				)
-				(hide yes)
-			)
-		)
-		(property "Value" "+3V3"
-			(at 95.25 81.28 0)
-			(effects
-				(font
-					(size 1.27 1.27)
-				)
-				(hide yes)
-			)
-		)
-		(property "Footprint" ""
-			(at 95.25 86.36 0)
-			(effects
-				(font
-					(size 1.27 1.27)
-				)
-				(hide yes)
-			)
-		)
-		(property "Datasheet" ""
-			(at 95.25 86.36 0)
-			(effects
-				(font
-					(size 1.27 1.27)
-				)
-				(hide yes)
-			)
-		)
-		(property "Description" "Power symbol creates a global label with name \"+3V3\""
-			(at 95.25 86.36 0)
-			(effects
-				(font
-					(size 1.27 1.27)
-				)
-				(hide yes)
-			)
-		)
-		(pin "1"
-		)
-		(instances
-			(project "Axis_MCU_V3"
-				(path "/73e46140-01b8-4ec1-93bb-0d72bea0e0ee"
-					(reference "#PWR027")
-					(unit 1)
-				)
-			)
-		)
-	)
-	(symbol
 		(lib_id "Project_Library:Pico")
 		(at 55.88 77.47 0)
@@
 					(unit 1)
 				)
+			)
+		)
+	)
+	(symbol
+		(lib_name "+3V3_1")
+		(lib_id "power:+3V3")
+		(at 95.25 86.36 0)
+		(unit 1)
+		(exclude_from_sim no)
+		(in_bom yes)
+		(on_board yes)
+		(dnp no)
+		(property "Reference" "#PWR027"
+			(at 95.25 90.17 0)
+			(effects
+				(font
+					(size 1.27 1.27)
+				)
+				(hide yes)
+			)
+		)
+		(property "Value" "+3V3"
+			(at 95.25 81.28 0)
+			(effects
+				(font
+					(size 1.27 1.27)
+				)
+			)
+		)
+		(property "Footprint" ""
+			(at 95.25 86.36 0)
+			(effects
+				(font
+					(size 1.27 1.27)
+				)
+				(hide yes)
+			)
+		)
+		(property "Datasheet" ""
+			(at 95.25 86.36 0)
+			(effects
+				(font
+					(size 1.27 1.27)
+				)
+				(hide yes)
+			)
+		)
+		(property "Description" "Power symbol creates a global label with name \"+3V3\""
+			(at 95.25 86.36 0)
+			(effects
+				(font
+					(size 1.27 1.27)
+				)
+				(hide yes)
+			)
+		)
+		(pin "1"
+		)
+		(instances
+			(project "Axis_MCU_V3"
+				(path "/73e46140-01b8-4ec1-93bb-0d72bea0e0ee"
+					(reference "#PWR027")
+					(unit 1)
+				)
