File: hardware/pcbs/Axis_MCU_V4/Axis_MCU_V4.kicad_sch (KiCad schematic)
At the start: 27 parts, among them J1 SWD, J2 GPIO, J3 UART, J4 HV_IDC, SW1 RES, U1 TCA9534, U2 Pico, U3 TCA9543A, U4 TCA9543A, U5 FM24CL16B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

Commit message: Add base board
Parts:
- BT1: now fitted
Connections:
- net I2C0_SCL: now also U2.7 (GPIO5), U3.12 (SCL); no longer U3.13 (SDA)
- net I2C0_SDA: now also U2.6 (GPIO4), U3.13 (SDA); no longer U3.12 (SCL)
- net I2C1_SCL: now also U2.5 (GPIO3), U4.12 (SCL); no longer U4.13 (SDA)
- net I2C1_SDA: now also U2.4 (GPIO2), U4.13 (SDA); no longer U4.12 (SCL)
- net RTC_CLK: now also U2.27 (GPIO21)
- net SPI0_A0: now also U2.19 (GPIO14)
- net SPI0_A1: now also U2.20 (GPIO15)
- net SPI0_MISO: now also U2.21 (GPIO16)
- net SPI0_SCK: now also U2.24 (GPIO18)
- net SPI1_A0: now also U2.9 (GPIO6)
- net SPI1_A1: now also U2.10 (GPIO7)
- net SPI1_MISO: now also U2.11 (GPIO8)
- net SPI1_MOSI: now also U2.15 (GPIO11), U2.25 (GPIO19)
- net SPI1_SCK: now also U2.14 (GPIO10)
- net UART_RX: now also U2.2 (GPIO1)
- net UART_TX: now also U2.1 (GPIO0)
- net ~{EXP0_INT}: now also U2.16 (GPIO12)
- net ~{EXP1_INT}: now also U2.17 (GPIO13)
- net ~{IO_INT}: now also U2.26 (GPIO20)
- net ~{SPI0_G}: now also U2.22 (GPIO17)
- net ~{SPI1_G}: now also U2.12 (GPIO9)
- net ~{TIMER_INT}: now also U2.29 (GPIO22)
Other:
- moved on the sheet: J1, J3
