File: hardware/pcbs/Axis_Base_Rev01/Axis_Base_Rev01.kicad_sch (KiCad schematic)
At the start: 17 parts, among them J1 SWD, J2 HV_IDC, J3 UART, SW1 RES, U1 DS3231MZ, U2 FM24CL16B, U3 Pico

Commit message: Changes
Parts:
- removed J2: HV_IDC, Connector_IDC:IDC-Header_2x04_P2.54mm_Vertical, symbol Connector_Generic:Conn_01x08
- removed J3: UART, Connector_JST:JST_SH_SM03B-SRSS-TB_1x03-1MP_P1.00mm_Horizontal, symbol Connector_Generic:Conn_01x03
- added C4, C5, C6, C7: 0.1u, Capacitor_SMD:C_0402_1005Metric, symbol Device:C_Small
- added D1: D_Small, symbol Device:D_Small
- added R3: 120, Resistor_SMD:R_0402_1005Metric, symbol Device:R_Small
- added R4: 1k, Resistor_SMD:R_0402_1005Metric, symbol Device:R_Small
- added R5: 1k, symbol Device:R_Small
- added U6: MCP25625-x-SS, Package_SO:SSOP-28_5.3x10.2mm_P0.65mm, symbol Interface_CAN_LIN:MCP25625-x-SS
- U3: footprint MCU_RaspberryPi_and_Boards:RPi_Pico_SMD_TH_No_Silkscreen -> RPi_Pico:RPi_Pico_SMD_TH
Connections:
- net +3V3: now also C4.1, C5.1, D1.1 (K), R4.1, U6.1 (VIO), U6.19 (VDD)
- net +5V: now also C6.1, U6.27 (VDDA)
- net GND: now also C4.2, C5.2, C6.2, C7.2, U6.10 (GND), U6.26 (VSS)
- net I2C1_SCL renamed I2C0_SCL
- net I2C1_SDA renamed I2C0_SDA
- new net: C7.1, D1.2 (A), R4.2, R5.1
- new net: R5.2, U6.18 (~{RESET})
- new net: U6.20 (TxCAN), U6.24 (TXD)
- new net: U6.21 (RxCAN), U6.28 (RXD)
- new net CANH: R3.1, U6.4 (CANH)
- new net CANL: R3.2, U6.3 (CANL)
- new net SPI0_MISO: U6.16 (SO)
- new net SPI0_MOSI: U6.15 (SI)
- new net SPI0_SCK: U6.14 (SCK)
- new net STBY: U6.5 (STBY)
- new net ~{CAN_INT}: U6.13 (~{INT})
- new net ~{Rx0BF}: U6.12 (~{Rx0BF})
- new net ~{Rx1BF}: U6.11 (~{Rx1BF})
- new net ~{SPI0_CS}: U6.17 (~{CS})
- new net ~{Tx0RTS}: U6.23 (~{Tx0RTS})
- new net ~{Tx1RTS}: U6.6 (~{Tx1RTS})
- new net ~{Tx2RTS}: U6.7 (~{Tx2RTS})
- no-connect marks 5 -> 4
Other:
- note added: "CAN Bus Controller/Interface"
- note added: "Capactor goes across +BATT"
- note added: "Config EEPROM/FRAM"
- note added: "I2C Address: 0b1101000"
- note removed: "EEPROM/FRAM"
- moved on the sheet: BT1, C1, C2, C3, H1, H2, H3, H4, J1, R1, R2, U1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
