File: hardware/pcbs/Axis_Base_Rev01/Axis_Base_Rev01.kicad_pcb (KiCad board)
At the start: 4 copper layers, 90 x 60 mm, 51 parts, among them J1 SWD, J10 HV_IDC, J2 GPIO, J3 Conn_01x04, J4 UART, J5 Conn_01x02, J7 EXT_SPI, J8 EXT_I2C, J9 GPIO, SW1 RES, U1 Pico, U2 ADS1119IPWR, U3 TCA9534, U4 MAX31855EASA, U5 PCA9544APWR, U7 MAX6107, U8 FM24CL16B, U9 DS3231MZ

Commit message: PCB updates
Parts:
- removed C10, C9: 0.1u, Capacitor_SMD:C_0402_1005Metric
- removed D1, D2: 4.7v, Package_TO_SOT_SMD:SOT-23
- removed J10: HV_IDC, Connector_IDC:IDC-Header_2x04_P2.54mm_Vertical
- removed J5: Conn_01x02, TerminalBlock_Phoenix:TerminalBlock_Phoenix_MKDS-1,5-2-5.08_1x02_P5.08mm_Horizontal
- removed J7: EXT_SPI, Connector_PinHeader_2.54mm:PinHeader_1x06_P2.54mm_Vertical
- removed J8: EXT_I2C, Connector_PinHeader_2.54mm:PinHeader_1x06_P2.54mm_Vertical
- removed J9: GPIO, Connector_PinHeader_2.54mm:PinHeader_1x08_P2.54mm_Vertical
- removed R10, R11, R12, R13, R14, R15, R16, R17, R18, R8, R9: 1k, Resistor_SMD:R_0402_1005Metric
- removed SW1: RES, Button_Switch_SMD:SW_SPST_B3U-1000P
- removed U7: MAX6107, Package_TO_SOT_SMD:SOT-23
- removed U8: FM24CL16B, Package_SO:SOIC-8_3.9x4.9mm_P1.27mm
- removed U9: DS3231MZ, Package_SO:SOIC-8_3.9x4.9mm_P1.27mm
- added BT1: BA2032, Footprints:BAT_BU2032SM-BT-GTR, F.Cu at (84.2, 57.0)
- added C6: 26p, Capacitor_SMD:C_0603_1608Metric, F.Cu at (107.2, 56.4)
- added Y1: ABM8G-20.000MHZ-18-D2Y-T, Footprints:Oscillator_Crystal_Abracon_SMD_ABM8G, F.Cu at (107.2, 53.6)
- C1, C2, C3, C4, C5, C8: footprint Capacitor_SMD:C_0402_1005Metric -> Capacitor_SMD:C_0603_1608Metric
- C7: value 0.1u -> 26p; footprint Capacitor_SMD:C_0402_1005Metric -> Capacitor_SMD:C_0603_1608Metric
- H1, H2, H3, H4: footprint MountingHole:MountingHole_2.7mm_M2.5 -> MountingHole:MountingHole_3.2mm_M3_Pad_Via
- J2: value GPIO -> CAN_1; footprint TerminalBlock_Phoenix:TerminalBlock_Phoenix_MKDS-1,5-8-5.08_1x08_P5.08mm_Horizontal -> Connector_JST:JST_PH_S4B-PH-SM4-TB_1x04-1MP_P2.00mm_Horizontal
- J3: value Conn_01x04 -> CAN_2; footprint TerminalBlock_Phoenix:TerminalBlock_Phoenix_MKDS-1,5-4-5.08_1x04_P5.08mm_Horizontal -> Connector_JST:JST_PH_S4B-PH-SM4-TB_1x04-1MP_P2.00mm_Horizontal
- J4: value UART -> CAN_3; footprint Connector_JST:JST_SH_SM03B-SRSS-TB_1x03-1MP_P1.00mm_Horizontal -> Connector_JST:JST_PH_S4B-PH-SM4-TB_1x04-1MP_P2.00mm_Horizontal
- R1, R2, R3, R4, R5, R6, R7: footprint Resistor_SMD:R_0402_1005Metric -> Resistor_SMD:R_0603_1608Metric
- U1: footprint MCU_RaspberryPi_and_Boards:RPi_Pico_SMD_TH_No_Silkscreen -> MCU_RaspberryPi_and_Boards:RPi_Pico_SMD_No_Silkscreen; moved to B.Cu
- U2: value ADS1119IPWR -> DS3231MZ; footprint Package_SO:TSSOP-16_4.4x5mm_P0.65mm -> Package_SO:SOIC-8_3.9x4.9mm_P1.27mm
- U3: value TCA9534 -> DS2411R; footprint Package_SO:TSSOP-16_4.4x5mm_P0.65mm -> Package_TO_SOT_SMD:SOT-23
- U4: value MAX31855EASA -> FM24CL16B
- U5: value PCA9544APWR -> MCP251863T-H; footprint Package_SO:TSSOP-20_4.4x6.5mm_P0.65mm -> Package_SO:SSOP-28_5.3x10.2mm_P0.65mm
- moved J4 72.8 mm to (134.7, 70.5), turned to 90 degrees
- moved C2 59.7 mm to (75.8, 85.4), turned to 0 degrees
- moved U2 51.8 mm to (75.8, 81.4)
- moved J2 50.2 mm to (119.2, 35.2), turned to 180 degrees
- moved U3 48.3 mm to (126.1, 78.1), turned to 0 degrees
- moved R3 47.2 mm to (125.8, 81.5), turned to 0 degrees
- moved C1 46.4 mm to (75.8, 77.4), turned to 0 degrees
- moved R7 41.7 mm to (85.4, 78.0), turned to 0 degrees
- moved C7 37.9 mm to (107.2, 50.8)
- moved C3 36.2 mm to (117.9, 74.2), turned to 0 degrees
- moved R5 32.8 mm to (118.4, 44.0), turned to 90 degrees
- moved R6 30.7 mm to (85.4, 81.2), turned to 0 degrees
- moved C5 25.7 mm to (119.2, 48.6), turned to 180 degrees
- moved C8 20.6 mm to (113.0, 61.6)
- moved C4 18.4 mm to (119.4, 61.6)
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Connections:
- C2 pad 1: +5V -> +BATT
- C7 pad 1: +3V3 -> Net-(U5-OSC1)
- C7 pad 2: GND -> Net-(C7-Pad2)
- J2 pad 1: +3V3 -> +5V
- J2 pad 2: /IO_1 -> /CANH
- J2 pad 3: /IO_2 -> /CANL
- J2 pad 4: /IO_3 -> GND
- J3 pad 2: /ADC_0 -> /CANH
- J3 pad 3: /ADC_1 -> /CANL
- J4 pad 1: /UART_RX -> +5V
- J4 pad 2: GND -> /CANH
- J4 pad 3: /UART_TX -> /CANL
- R1 pad 2: /I2C0_SDA -> /RTC_CLK
- R2 pad 2: /I2C0_SCL -> /~{TIMER_INT}
- R3 pad 2: /~{IO_INT} -> Net-(U3-I/O)
- R4 pad 1: +3V3 -> Net-(U3-I/O)
- R4 pad 2: /I2C1_SCL -> /1WIRE
- R5 pad 1: +3V3 -> /CANH
- R5 pad 2: /I2C1_SDA -> /CANL
- R6 pad 2: /~{MUX_INT} -> /I2C0_SDA
- R7 pad 2: /ADS_SDA -> /I2C0_SCL
- U1 pad 1: /UART_TX -> /SPI0_MISO
- U1 pad 10: /GPIO7 -> /STBY
- U1 pad 11: /SPI1_RX -> unconnected-(U1-GPIO8-Pad11)
- U1 pad 12: /~{SPI1_CS0} -> unconnected-(U1-GPIO9-Pad12)
- U1 pad 14: /SPI1_SCK -> unconnected-(U1-GPIO10-Pad14)
- U1 pad 15: /SPI1_TX -> unconnected-(U1-GPIO11-Pad15)
- U1 pad 16: /I2C0_SDA -> unconnected-(U1-GPIO12-Pad16)
- U1 pad 17: /I2C0_SCL -> unconnected-(U1-GPIO13-Pad17)
- U1 pad 19: /~{IO_INT} -> unconnected-(U1-GPIO14-Pad19)
- U1 pad 2: /UART_RX -> /~{SPI0_CS}
- U1 pad 20: /~{SPI0_CS1} -> unconnected-(U1-GPIO15-Pad20)
- U1 pad 21: /SPI0_RX -> /I2C0_SDA
- U1 pad 22: /~{SPI0_CS0} -> /I2C0_SCL
- U1 pad 24: /SPI0_SCK -> /RTC_CLK
- U1 pad 25: unconnected-(U1-GPIO19-Pad25)_0 -> /~{TIMER_INT}
- U1 pad 26: /HV_IO1 -> /1WIRE
- U1 pad 27: /ZC_SIG -> unconnected-(U1-GPIO21-Pad27)
- U1 pad 29: /~{MUX_INT} -> unconnected-(U1-GPIO22-Pad29)
- U1 pad 30: Net-(U1-RUN) -> unconnected-(U1-RUN-Pad30)
- U1 pad 31: /I2C1_SDA -> unconnected-(U1-GPIO26_ADC0-Pad31)
- U1 pad 32: /I2C1_SCL -> unconnected-(U1-GPIO27_ADC1-Pad32)
- U1 pad 34: /HV_IO2 -> unconnected-(U1-GPIO28_ADC2-Pad34)
- U1 pad 4: /GPIO2 -> /SPI0_SCK
- U1 pad 5: /GPIO3 -> /SPI0_MOSI
- U1 pad 6: /GPIO4 -> /~{nINT}
- U1 pad 7: /GPIO5 -> /~{nINT1}
- U1 pad 9: /GPIO6 -> /~{nINT2}
- U2 pad 1: GND -> /RTC_CLK
- U2 pad 2: GND -> +3V3
- U2 pad 3: +3V3 -> /~{TIMER_INT}
- U2 pad 4: GND -> unconnected-(U2-~{RST}-Pad4)
- U2 pad 6: unconnected-(U2-AIN3-Pad6) -> +BATT
- U2 pad 7: unconnected-(U2-AIN2-Pad7) -> /I2C0_SDA
- U2 pad 8: GND -> /I2C0_SCL
- U3 pad 1: GND -> Net-(U3-I/O)
- U3 pad 2: GND -> +3V3
- U4 pad 1: GND -> unconnected-(U4-Pad1)
- U4 pad 2: /THCPL1_NEG -> unconnected-(U4-Pad2)
- U4 pad 3: /THCPL1_POS -> unconnected-(U4-Pad3)
- U4 pad 4: +3V3 -> GND
- U4 pad 5: /SPI0_SCK -> /I2C0_SDA
- U4 pad 6: /~{SPI0_CS0} -> /I2C0_SCL
- U4 pad 7: /SPI0_RX -> GND
- U4 pad 8: (no net) -> +3V3
- U5 pad 1: GND -> +3V3
- U5 pad 10: GND -> /SPI0_MOSI
- U5 pad 11: /~{EXT_INT} -> /SPI0_MISO
- U5 pad 12: /EXT_SDA -> (no net)
- U5 pad 13: /EXT_SCL -> /~{SPI0_CS}
- U5 pad 14: /~{INT_3} -> +3V3
- U5 pad 15: /HV_SDA -> Net-(U5-TXD)
- U5 pad 16: /HV_SCL -> Net-(U5-RXD)
- U5 pad 17: /~{MUX_INT} -> (no net)
- U5 pad 18: /I2C1_SCL -> unconnected-(U5-CLKOUT-Pad18)
- U5 pad 19: /I2C1_SDA -> /~{nINT}
- U5 pad 2: GND -> (no net)
- U5 pad 20: +3V3 -> Net-(U5-OSC2)
- U5 pad 3: GND -> /CANL
- U5 pad 4: /~{TIMER_INT} -> /CANH
- U5 pad 5: /TIMER_SDA -> /STBY
- U5 pad 6: /TIMER_SCL -> /~{nINT1}
- U5 pad 7: /~{ADS_RDY} -> /~{nINT2}
- U5 pad 8: /ADS_SDA -> (no net)
- U5 pad 9: /ADS_SCL -> /SPI0_SCK
Routing:
- net +3V3: track 241.1 -> 0.00 mm, vias 18 -> 0
- net /SWDIO: track 107.7 -> 0.00 mm
- net /SWCLK: track 95.4 -> 0.00 mm
- net +5V: track 83.7 -> 0.00 mm
- net /I2C1_SCL: track 74.4 -> 0.00 mm, vias 2 -> 0
- net /I2C1_SDA: track 66.7 -> 0.00 mm, vias 2 -> 0
- net /HV_SCL: track 55.4 -> 0.00 mm, vias 3 -> 0
- net /HV_IO1: track 53.0 -> 0.00 mm, vias 2 -> 0
- net /HV_SDA: track 51.4 -> 0.00 mm, vias 1 -> 0
- net /ZC_SIG: track 45.4 -> 0.00 mm, vias 2 -> 0
- net GND: track 41.5 -> 0.00 mm, vias 45 -> 0
- net /~{MUX_INT}: track 35.8 -> 0.00 mm, vias 1 -> 0
- net /EXT_SCL: track 35.6 -> 0.00 mm, vias 1 -> 0
- net Net-(U1-RUN): track 33.3 -> 0.00 mm, vias 2 -> 0
- net /I2C0_SDA: track 31.3 -> 0.00 mm, vias 2 -> 0
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- removed copper zone on In2.Cu, net +3V3
- removed copper zone on B.Cu, net GND
- removed copper zone on F.Cu, net GND
- removed copper zone on In1.Cu, net GND
Other:
- board outline removed
- board text removed: "+"
- board text removed: "+5v"
- board text removed: "-"
- board text removed: "1"
- board text removed: "2"
- board text removed: "3"
- board text removed: "3v3"
- board text removed: "ADC0"
- board text removed: "ADC1"
- board text removed: "Axis PCB V2 Rev. 2 Meigs2"
- board text removed: "GND"
- board text removed: "HV Breakout"
- board text removed: "M3"
- board text removed: "WayWayWay"
